File: hardware/midi2cv.kicad_pcb (KiCad board)
At the start: 2 copper layers, 0 parts

Commit message: First preliminary board design
Parts:
- added C1: 100n, Capacitor_SMD:C_0603_1608Metric, F.Cu at (96.4, 75.4)
- added C10: 100n, Capacitor_SMD:C_0603_1608Metric, F.Cu at (93.1, 61.8)
- added C11: 4.7u, Capacitor_SMD:C_0603_1608Metric, F.Cu at (79.2, 73.8)
- added C12: 100n, Capacitor_SMD:C_0603_1608Metric, F.Cu at (87.5, 61.2)
- added C13: 100n, Capacitor_SMD:C_0603_1608Metric, F.Cu at (95.2, 66.5)
- added C14: 100n, Capacitor_SMD:C_0603_1608Metric, F.Cu at (93.9, 76.3)
- added C15: 100n, Capacitor_SMD:C_0603_1608Metric, F.Cu at (81.3, 76.3)
- added C16: 100n, Capacitor_SMD:C_0603_1608Metric, F.Cu at (80.0, 66.5)
- added C17: 100n, Capacitor_SMD:C_0603_1608Metric, F.Cu at (82.9, 82.4)
- added C18: 100n, Capacitor_SMD:C_0603_1608Metric, F.Cu at (82.9, 85.5)
- added C19: 3.3u, Capacitor_SMD:C_0603_1608Metric, F.Cu at (82.9, 83.9)
- added C2: 100n, Capacitor_SMD:C_0603_1608Metric, F.Cu at (81.0, 43.5)
- added C20: 220n, Capacitor_SMD:C_0603_1608Metric, F.Cu at (87.0, 89.1)
- added C21: 100n, Capacitor_SMD:C_0603_1608Metric, F.Cu at (81.5, 101.0)
- added C22: 100n, Capacitor_SMD:C_0603_1608Metric, F.Cu at (94.2, 101.0)
- added C23: 22p, Capacitor_SMD:C_0603_1608Metric, F.Cu at (84.8, 96.4)
- added C24: 22p, Capacitor_SMD:C_0603_1608Metric, F.Cu at (90.9, 96.4)
- added C25: 22p, Capacitor_SMD:C_0603_1608Metric, F.Cu at (84.8, 105.5)
- added C26: 22p, Capacitor_SMD:C_0603_1608Metric, F.Cu at (90.9, 105.5)
- added C27: 100n, Capacitor_SMD:C_0603_1608Metric, F.Cu at (94.9, 90.1)
- added C28: 100n, Capacitor_SMD:C_0603_1608Metric, F.Cu at (100.5, 97.5)
- added C29: 3.3u, Capacitor_SMD:C_0603_1608Metric, F.Cu at (96.4, 90.1)
- added C3: 100n, Capacitor_SMD:C_0603_1608Metric, F.Cu at (98.9, 44.8)
- added C30: 100n, Capacitor_SMD:C_0603_1608Metric, F.Cu at (113.2, 97.6)
- added C31: 100n, Capacitor_SMD:C_0603_1608Metric, F.Cu at (100.5, 111.8)
- added C32: 1u, Capacitor_SMD:C_0603_1608Metric, F.Cu at (102.2, 87.8)
- added C33: 100n, Capacitor_SMD:C_0603_1608Metric, F.Cu at (102.2, 86.2)
- added C34: 100n, Capacitor_SMD:C_0603_1608Metric, F.Cu at (113.2, 112.3)
- added C35: 10p, Capacitor_SMD:C_0603_1608Metric, F.Cu at (103.8, 93.0)
- added C36: 10p, Capacitor_SMD:C_0603_1608Metric, F.Cu at (103.8, 102.1)
- added C37: 10p, Capacitor_SMD:C_0603_1608Metric, F.Cu at (109.9, 102.1)
- added C38: 10p, Capacitor_SMD:C_0603_1608Metric, F.Cu at (109.9, 93.0)
- added C39: 10p, Capacitor_SMD:C_0603_1608Metric, F.Cu at (103.8, 107.2)
- added C4: 1u, Capacitor_SMD:C_0603_1608Metric, F.Cu at (86.1, 43.5)
- added C40: 10p, Capacitor_SMD:C_0603_1608Metric, F.Cu at (103.8, 116.3)
- added C41: 10p, Capacitor_SMD:C_0603_1608Metric, F.Cu at (109.9, 116.3)
- added C42: 10p, Capacitor_SMD:C_0603_1608Metric, F.Cu at (109.9, 107.2)
- added C43: 10u, Capacitor_SMD:C_0805_2012Metric, F.Cu at (107.6, 63.8)
- added C44: 10u, Capacitor_SMD:C_0805_2012Metric, F.Cu at (113.2, 60.8)
- added C45: 100n, Capacitor_SMD:C_0603_1608Metric, F.Cu at (98.9, 62.0)
- added C46: 10u, Capacitor_SMD:C_0805_2012Metric, F.Cu at (99.0, 59.9)
- added C47: 100n, Capacitor_SMD:C_0603_1608Metric, F.Cu at (106.3, 60.7)
- added C48: 22u, Capacitor_SMD:C_0805_2012Metric, F.Cu at (109.3, 88.1)
- added C49: 22u, Capacitor_SMD:C_0805_2012Metric, F.Cu at (110.4, 64.5)
- added C5: 100n, Capacitor_SMD:C_0603_1608Metric, F.Cu at (79.2, 118.0)
- added C50: 22u, Capacitor_SMD:C_0805_2012Metric, F.Cu at (108.3, 60.7)
- added C51: 1u, Capacitor_SMD:C_0603_1608Metric, F.Cu at (114.2, 46.9)
- added C52: 1u, Capacitor_SMD:C_0603_1608Metric, F.Cu at (103.3, 60.1)
- added C53: 1u, Capacitor_SMD:C_0603_1608Metric, F.Cu at (108.9, 47.6)
- added C54: 1u, Capacitor_SMD:C_0603_1608Metric, F.Cu at (102.5, 66.7)
- added C55: 100p, Capacitor_SMD:C_0603_1608Metric, F.Cu at (105.2, 34.2)
- added C56: 100p, Capacitor_SMD:C_0603_1608Metric, F.Cu at (113.5, 37.5)
- added C57: 100n, Capacitor_SMD:C_0603_1608Metric, F.Cu at (106.9, 42.2)
- added C6: 27p, Capacitor_SMD:C_0603_1608Metric, F.Cu at (93.1, 60.3)
- added C7: 1u, Capacitor_SMD:C_0603_1608Metric, F.Cu at (83.8, 61.2)
- added C8: 27p, Capacitor_SMD:C_0603_1608Metric, F.Cu at (89.9, 60.3)
- added C9: 100n, Capacitor_SMD:C_0603_1608Metric, F.Cu at (85.3, 61.2)
- added D1: BAT54S, Package_TO_SOT_SMD:SOT-23, F.Cu at (53.8, 34.4)
- added D2: 1N4148, Diode_SMD:D_SOD-123, F.Cu at (95.1, 30.7)
- added D3: 1N5819, Diode_SMD:D_SOD-123, F.Cu at (110.7, 84.8)
- added D4: 1N5819, Diode_SMD:D_SOD-123, F.Cu at (110.7, 68.8)
- added D5: B72500D0160H060, Diode_SMD:D_0603_1608Metric, F.Cu at (109.7, 34.2)
- added D6: B72500D0160H060, Diode_SMD:D_0603_1608Metric, F.Cu at (113.5, 32.9)
- added FB1: 100 @ 100MHz, Inductor_SMD:L_0805_2012Metric, F.Cu at (112.1, 88.1)
- added FB2: 100 @ 100MHz, Inductor_SMD:L_0805_2012Metric, F.Cu at (112.4, 64.5)
- added IC1: SN74AHCT244PW, SN74AHCT244PW:SOP65P640X120-20N, F.Cu at (84.3, 114.0)
- added IC2: LP5012PWR, LP5012PWR:SOP65P640X120-24N, F.Cu at (82.8, 37.9)
- added IC3: DAC8564IAPW, DAC5578:SOP65P640X120-16N, F.Cu at (87.1, 84.5)
- added IC4: DAC5578SPWR, DAC5578:SOP65P640X120-16N, F.Cu at (97.9, 84.6)
- added IC5: ADP150AUJZ-3.3-R7, ADP150AUJZ-3.3-R7:SOT95P280X100-5N, F.Cu at (102.2, 63.4)
- added J1: Conn_02x06_Odd_Even, Connector_PinSocket_2.54mm:PinSocket_2x06_P2.54mm_Vertical, F.Cu at (90.8, 29.8)
- added J10, J11: PJ398SM, Connector_Audio:Jack_3.5mm_QingPu_WQP-PJ398SM_Vertical_CircularHoles, B.Cu at (69.2, 91.4)
- added J12: PJ398SM, Connector_Audio:Jack_3.5mm_QingPu_WQP-PJ398SM_Vertical_CircularHoles, B.Cu at (69.2, 117.2)
- added J13: PJ398SM, Connector_Audio:Jack_3.5mm_QingPu_WQP-PJ398SM_Vertical_CircularHoles, B.Cu at (68.8, 43.4)
- added J14, J15: PJ398SM, Connector_Audio:Jack_3.5mm_QingPu_WQP-PJ398SM_Vertical_CircularHoles, B.Cu at (59.4, 65.7)
- added J16, J17: PJ398SM, Connector_Audio:Jack_3.5mm_QingPu_WQP-PJ398SM_Vertical_CircularHoles, B.Cu at (59.4, 91.4)
- added J18: PJ398SM, Connector_Audio:Jack_3.5mm_QingPu_WQP-PJ398SM_Vertical_CircularHoles, B.Cu at (59.4, 117.2)
- added J19: PJ398SM, Connector_Audio:Jack_3.5mm_QingPu_WQP-PJ398SM_Vertical_CircularHoles, B.Cu at (40.1, 43.4)
- added J2: Conn_02x06_Odd_Even, Connector_PinSocket_2.54mm:PinSocket_2x06_P2.54mm_Vertical, F.Cu at (113.7, 29.8)
- added J20, J21: PJ398SM, Connector_Audio:Jack_3.5mm_QingPu_WQP-PJ398SM_Vertical_CircularHoles, B.Cu at (49.5, 65.7)
- added J22, J23: PJ398SM, Connector_Audio:Jack_3.5mm_QingPu_WQP-PJ398SM_Vertical_CircularHoles, B.Cu at (49.5, 91.4)
- added J24: PJ398SM, Connector_Audio:Jack_3.5mm_QingPu_WQP-PJ398SM_Vertical_CircularHoles, B.Cu at (49.5, 117.2)
- added J25, J26: PJ398SM, Connector_Audio:Jack_3.5mm_QingPu_WQP-PJ398SM_Vertical_CircularHoles, B.Cu at (39.8, 65.7)
- added J27, J28: PJ398SM, Connector_Audio:Jack_3.5mm_QingPu_WQP-PJ398SM_Vertical_CircularHoles, B.Cu at (39.8, 91.4)
- added J29: PJ398SM, Connector_Audio:Jack_3.5mm_QingPu_WQP-PJ398SM_Vertical_CircularHoles, B.Cu at (39.8, 117.2)
- added J3: Conn_02x10_Odd_Even, Connector_PinSocket_2.54mm:PinSocket_2x12_P2.54mm_Vertical, F.Cu at (109.9, 122.6)
- added J30: Conn_02x05_Odd_Even, Connector_PinHeader_1.27mm:PinHeader_2x05_P1.27mm_Vertical, B.Cu at (80.0, 61.5)
- added J31: Eurorack PWR, Connector_IDC:IDC-Header_2x05_P2.54mm_Vertical, B.Cu at (109.1, 82.2)
- added J4: Conn_02x06_Odd_Even, Connector_PinHeader_2.54mm:PinHeader_2x06_P2.54mm_Vertical, F.Cu at (59.6, 29.8)
- added J5: Conn_02x06_Odd_Even, Connector_PinHeader_2.54mm:PinHeader_2x06_P2.54mm_Vertical, F.Cu at (36.7, 29.8)
- added J6: Conn_02x10_Odd_Even, Connector_PinHeader_2.54mm:PinHeader_2x12_P2.54mm_Vertical, F.Cu at (68.5, 120.0)
- added J7: SD-50BV, SD-50BV:SD-50BV, B.Cu at (54.5, 34.3)
- added J8, J9: PJ398SM, Connector_Audio:Jack_3.5mm_QingPu_WQP-PJ398SM_Vertical_CircularHoles, B.Cu at (69.2, 65.7)
- added L1: 10u, Inductor_SMD:L_0805_2012Metric, F.Cu at (110.6, 60.7)
- added R1: 100k, Resistor_SMD:R_0603_1608Metric, F.Cu at (57.3, 35.9)
- added R10: 36k, Resistor_SMD:R_0603_1608Metric, F.Cu at (87.0, 92.1)
- added R11: 33k, Resistor_SMD:R_0603_1608Metric, F.Cu at (82.2, 98.2)
- added R12: 33k, Resistor_SMD:R_0603_1608Metric, F.Cu at (93.4, 98.2)
- added R13: 33k, Resistor_SMD:R_0603_1608Metric, F.Cu at (82.2, 103.8)
- added R14: 33k, Resistor_SMD:R_0603_1608Metric, F.Cu at (93.4, 103.8)
- added R15: 180k, Resistor_SMD:R_0603_1608Metric, F.Cu at (82.2, 96.6)
- added R16: 180k, Resistor_SMD:R_0603_1608Metric, F.Cu at (93.4, 96.6)
- added R17: 180k, Resistor_SMD:R_0603_1608Metric, F.Cu at (82.2, 105.3)
- added R18: 180k, Resistor_SMD:R_0603_1608Metric, F.Cu at (93.4, 105.3)
- added R19: 1k, Resistor_SMD:R_0603_1608Metric, F.Cu at (86.3, 96.4)
- added R2: 100k, Resistor_SMD:R_0603_1608Metric, F.Cu at (54.0, 37.1)
- added R20: 1k, Resistor_SMD:R_0603_1608Metric, F.Cu at (89.3, 96.4)
- added R21: 1k, Resistor_SMD:R_0603_1608Metric, F.Cu at (86.3, 105.5)
- added R22: 1k, Resistor_SMD:R_0603_1608Metric, F.Cu at (89.3, 105.5)
- added R23: 33k, Resistor_SMD:R_0603_1608Metric, F.Cu at (102.2, 84.7)
- added R24: 22k, Resistor_SMD:R_0603_1608Metric, F.Cu at (102.2, 83.2)
- added R25: 10k, Resistor_SMD:R_0603_1608Metric, F.Cu at (102.2, 81.7)
- added R26: 36k, Resistor_SMD:R_0603_1608Metric, F.Cu at (101.2, 94.7)
- added R27: 36k, Resistor_SMD:R_0603_1608Metric, F.Cu at (101.2, 100.3)
- added R28: 36k, Resistor_SMD:R_0603_1608Metric, F.Cu at (112.4, 100.3)
- added R29: 36k, Resistor_SMD:R_0603_1608Metric, F.Cu at (112.4, 94.7)
- added R3: 27k, Resistor_SMD:R_0603_1608Metric_Pad0.98x0.95mm_HandSolder, F.Cu at (84.3, 43.5)
- added R30: 150k, Resistor_SMD:R_0603_1608Metric, F.Cu at (101.2, 93.2)
- added R31: 150k, Resistor_SMD:R_0603_1608Metric, F.Cu at (101.2, 101.9)
- added R32: 150k, Resistor_SMD:R_0603_1608Metric, F.Cu at (112.4, 101.9)
- added R33: 150k, Resistor_SMD:R_0603_1608Metric, F.Cu at (112.4, 93.2)
- added R34: 1k, Resistor_SMD:R_0603_1608Metric, F.Cu at (105.3, 93.0)
- added R35: 1k, Resistor_SMD:R_0603_1608Metric, F.Cu at (105.3, 102.1)
- added R36: 1k, Resistor_SMD:R_0603_1608Metric, F.Cu at (108.3, 102.1)
- added R37: 1k, Resistor_SMD:R_0603_1608Metric, F.Cu at (108.3, 93.0)
- added R38: 36k, Resistor_SMD:R_0603_1608Metric, F.Cu at (101.2, 109.0)
- added R39: 36k, Resistor_SMD:R_0603_1608Metric, F.Cu at (101.2, 114.6)
- added R4: 10k, Resistor_SMD:R_0603_1608Metric, F.Cu at (82.5, 43.5)
- added R40: 36k, Resistor_SMD:R_0603_1608Metric, F.Cu at (112.4, 114.6)
- added R41: 36k, Resistor_SMD:R_0603_1608Metric, F.Cu at (112.4, 109.0)
- added R42: 150k, Resistor_SMD:R_0603_1608Metric, F.Cu at (101.2, 107.4)
- added R43: 150k, Resistor_SMD:R_0603_1608Metric, F.Cu at (101.2, 116.1)
- added R44: 150k, Resistor_SMD:R_0603_1608Metric, F.Cu at (112.4, 116.1)
- added R45: 150k, Resistor_SMD:R_0603_1608Metric, F.Cu at (112.4, 107.4)
- added R46: 1k, Resistor_SMD:R_0603_1608Metric, F.Cu at (105.3, 107.2)
- added R47: 1k, Resistor_SMD:R_0603_1608Metric, F.Cu at (105.3, 116.3)
- added R48: 1k, Resistor_SMD:R_0603_1608Metric, F.Cu at (108.3, 116.3)
- added R49: 1k, Resistor_SMD:R_0603_1608Metric, F.Cu at (108.3, 107.2)
- added R5: 220R, Resistor_SMD:R_0603_1608Metric, F.Cu at (96.0, 28.7)
- added R50: 1k8, Resistor_SMD:R_0603_1608Metric, F.Cu at (112.0, 47.6)
- added R51: 140k, Resistor_SMD:R_0603_1608Metric, F.Cu at (108.2, 34.2)
- added R52: 140k, Resistor_SMD:R_0603_1608Metric, F.Cu at (113.5, 34.5)
- added R53: 200k, Resistor_SMD:R_0603_1608Metric, F.Cu at (106.9, 43.8)
- added R54: 200k, Resistor_SMD:R_0603_1608Metric, F.Cu at (112.8, 41.4)
- added R55: 33k, Resistor_SMD:R_0603_1608Metric, F.Cu at (106.7, 34.2)
- added R56: 33k, Resistor_SMD:R_0603_1608Metric, F.Cu at (113.5, 36.0)
- added R57: 100R, Resistor_SMD:R_0603_1608Metric, F.Cu at (103.6, 35.8)
- added R58: 100R, Resistor_SMD:R_0603_1608Metric, F.Cu at (113.5, 39.1)
- added R6: 10k, Resistor_SMD:R_0603_1608Metric, F.Cu at (95.9, 44.8)
- added R7: 680R, Resistor_SMD:R_0603_1608Metric, F.Cu at (89.9, 61.8)
- added R8: 10k, Resistor_SMD:R_0603_1608Metric, F.Cu at (96.7, 66.5)
- added R9: 33k, Resistor_SMD:R_0603_1608Metric, F.Cu at (87.0, 90.6)
- added S1: TC002-N11AS1XKT-RGB, TC002-N11AS1XKT-RGB:TC002N11AS1XKTRGB, B.Cu at (71.0, 51.7)
- added S2: TC002-N11AS1XKT-RGB, TC002-N11AS1XKT-RGB:TC002N11AS1XKTRGB, B.Cu at (61.5, 51.7)
- added S3: TC002-N11AS1XKT-RGB, TC002-N11AS1XKT-RGB:TC002N11AS1XKTRGB, B.Cu at (51.9, 51.7)
- added S4: TC002-N11AS1XKT-RGB, TC002-N11AS1XKT-RGB:TC002N11AS1XKTRGB, B.Cu at (42.4, 51.7)
- added U1: AT24C256C, Package_SO:SOIC-8_3.9x4.9mm_P1.27mm, F.Cu at (101.0, 74.2)
- added U10: MCP6002-xMS, Package_SO:SOIC-8_3.9x4.9mm_P1.27mm, F.Cu at (108.1, 38.5)
- added U2: 6N137, Package_DIP:SMDIP-8_W9.53mm, F.Cu at (95.1, 38.0)
- added U3: STM32F401RBTx, Package_QFP:LQFP-64_10x10mm_P0.5mm, F.Cu at (87.5, 70.2)
- added U4: OPA4172, Package_SO:TSSOP-14_4.4x5mm_P0.65mm, F.Cu at (87.8, 101.0)
- added U5: TL074, Package_SO:TSSOP-14_4.4x5mm_P0.65mm, F.Cu at (106.8, 97.5)
- added U6: TL074, Package_SO:TSSOP-14_4.4x5mm_P0.65mm, F.Cu at (106.8, 111.8)
- added U7: LM1117-3.3, Package_TO_SOT_SMD:SOT-223, F.Cu at (100.5, 54.2)
- added U8: LM1117-5.0, Package_TO_SOT_SMD:SOT-223, F.Cu at (109.6, 54.2)
- added U9: LM4040DBZ-10, Package_TO_SOT_SMD:SOT-23, F.Cu at (111.0, 44.7)
- added Y1: X50328MSB2GI, Crystal:Crystal_SMD_5032-2Pin_5.0x3.2mm, F.Cu at (91.4, 57.5)
- added mouse-bite-2mm-slot: VAL**, Panelization:mouse-bite-2mm-slot, F.Cu at (75.2, 119.9)
- added mouse-bite-2mm-slot: VAL**, Panelization:mouse-bite-2mm-slot, F.Cu at (75.2, 67.1)
- added mouse-bite-2mm-slot: VAL**, Panelization:mouse-bite-2mm-slot, F.Cu at (75.2, 51.1)
- added mouse-bite-2mm-slot: VAL**, Panelization:mouse-bite-2mm-slot, F.Cu at (75.2, 30.7)
Routing:
- net +3V3: track 0.00 -> 295.7 mm, vias 0 -> 9
- net GND: track 0.00 -> 150.9 mm, vias 0 -> 116
- net +5V: track 0.00 -> 134.7 mm
- net VEE: track 0.00 -> 111.4 mm, vias 0 -> 4
- net +3.3VA: track 0.00 -> 97.6 mm, vias 0 -> 6
- net VCC: track 0.00 -> 93.2 mm, vias 0 -> 5
- net dac8_out_b_front: track 0.00 -> 90.8 mm
- net var_out_front: track 0.00 -> 78.0 mm
- net clock_out_front: track 0.00 -> 75.5 mm, vias 0 -> 2
- net dac8_out_a_front: track 0.00 -> 74.8 mm
- net dac4_out_b_front: track 0.00 -> 74.5 mm
- net dac8_out_c_front: track 0.00 -> 72.8 mm
- net run_out_front: track 0.00 -> 72.4 mm, vias 0 -> 2
- net led_out_d_g_front: track 0.00 -> 71.0 mm
- net 1_16_out_front: track 0.00 -> 69.4 mm
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- added copper zone on B.Cu, net GND
- added copper zone on F.Cu, net GND
Other:
- board outline added: 80.8 x 99.1 mm
- net class Power added: clearance 0.2, trace_width 0.4, via_dia 0.8, via_drill 0.5

Commit message: Layed out stretched design
Parts:
- removed the J10 at (69.2, 91.4)
- removed the J15 at (59.4, 65.7)
- removed the J16 at (59.4, 91.4)
- removed the J21 at (49.5, 65.7)
- removed the J22 at (49.5, 91.4)
- removed the J26 at (39.8, 65.7)
- removed the J27 at (39.8, 91.4)
- removed the J31 at (109.1, 82.2)
- removed the J6 at (68.5, 120.0)
- removed the J9 at (69.2, 65.7)
- removed the mouse-bite-2mm-slot at (75.2, 119.9)
- removed the mouse-bite-2mm-slot at (75.2, 67.1)
- removed the mouse-bite-2mm-slot at (75.2, 30.7)
- added J13: PJ398SM, Connector_Audio:Jack_3.5mm_QingPu_WQP-PJ398SM_Vertical_CircularHoles, B.Cu at (69.2, 104.1)
- added J14: PJ398SM, Connector_Audio:Jack_3.5mm_QingPu_WQP-PJ398SM_Vertical_CircularHoles, B.Cu at (69.2, 133.1)
- added J19: PJ398SM, Connector_Audio:Jack_3.5mm_QingPu_WQP-PJ398SM_Vertical_CircularHoles, B.Cu at (59.4, 104.1)
- added J20: PJ398SM, Connector_Audio:Jack_3.5mm_QingPu_WQP-PJ398SM_Vertical_CircularHoles, B.Cu at (59.4, 133.1)
- added J24: PJ398SM, Connector_Audio:Jack_3.5mm_QingPu_WQP-PJ398SM_Vertical_CircularHoles, B.Cu at (49.5, 101.1)
- added J25: PJ398SM, Connector_Audio:Jack_3.5mm_QingPu_WQP-PJ398SM_Vertical_CircularHoles, B.Cu at (49.5, 104.1)
- added J29: PJ398SM, Connector_Audio:Jack_3.5mm_QingPu_WQP-PJ398SM_Vertical_CircularHoles, B.Cu at (39.8, 101.1)
- added J32: Conn_02x05_Odd_Even, Connector_PinHeader_1.27mm:PinHeader_2x05_P1.27mm_Vertical, B.Cu at (80.6, 53.3)
- added J33: Eurorack PWR, Connector_IDC:IDC-Header_2x05_P2.54mm_Vertical, B.Cu at (109.4, 130.2)
- added J4: Conn_01x12, Connector_PinSocket_2.54mm:PinSocket_1x12_P2.54mm_Vertical, F.Cu at (109.8, 118.6)
- added J7: Conn_01x10, Connector_PinHeader_2.54mm:PinHeader_1x10_P2.54mm_Vertical, F.Cu at (43.1, 86.6)
- added J8: Conn_01x12, Connector_PinHeader_2.54mm:PinHeader_1x12_P2.54mm_Vertical, F.Cu at (40.5, 118.6)
- added mouse-bite-2mm-slot: VAL**, Panelization:mouse-bite-2mm-slot, F.Cu at (75.2, 127.3)
- added mouse-bite-2mm-slot: VAL**, Panelization:mouse-bite-2mm-slot, F.Cu at (75.2, 109.1)
- added mouse-bite-2mm-slot: VAL**, Panelization:mouse-bite-2mm-slot, F.Cu at (75.2, 30.6)
- J3: value Conn_02x10_Odd_Even -> Conn_01x10; footprint Connector_PinSocket_2.54mm:PinSocket_2x12_P2.54mm_Vertical -> Connector_PinSocket_2.54mm:PinSocket_1x10_P2.54mm_Vertical
- J30: value Conn_02x05_Odd_Even -> PJ398SM; footprint Connector_PinHeader_1.27mm:PinHeader_2x05_P1.27mm_Vertical -> Connector_Audio:Jack_3.5mm_QingPu_WQP-PJ398SM_Vertical_CircularHoles
- moved U7 77.4 mm to (80.5, 129.0), turned to 270 degrees
- moved U8 77.4 mm to (90.4, 129.2), turned to 270 degrees
- moved C50 72.6 mm to (85.5, 129.6)
- moved C47 68.7 mm to (85.5, 126.2), turned to 90 degrees
- moved C44 66.9 mm to (87.1, 122.4), turned to 0 degrees
- moved C46 65.3 mm to (80.3, 122.4)
- moved L1 64.8 mm to (90.8, 122.4), turned to 180 degrees
- moved FB2 63.9 mm to (96.5, 126.4)
- moved D4 63.7 mm to (96.5, 130.9), turned to 270 degrees
- moved C52 62.4 mm to (102.3, 122.4)
- moved C45 62.3 mm to (83.7, 122.4), turned to 0 degrees
- moved C43 60.0 mm to (94.8, 122.4)
- moved IC5 59.3 mm to (106.4, 122.6), turned to 0 degrees
- moved C49 59.1 mm to (98.5, 122.4), turned to 180 degrees
- moved J30 58.7 mm to (39.8, 104.1), turned to 180 degrees
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- renumbered J8 to J10, J13 to J15, J14 to J16, J19 to J21, J20 to J22, J24 to J26, J25 to J27, J29 to J31, J4 to J5, J5 to J6, J7 to J9
Connections:
- J11 pad T: dac4_out_c_front -> dac4_out_a_front
- J12 pad T: dac4_out_d_front -> dac4_out_b_front
- J17 pad T: gate_out_c_front -> gate_out_a_front
- J18 pad T: gate_out_d_front -> gate_out_b_front
- J23 pad T: dac8_out_e_front -> dac8_out_a_front
- J28 pad T: dac8_out_f_front -> dac8_out_b_front
- J3 pad 1: dac8_out_g_back -> GND
- J3 pad 10: dac4_out_d_back -> GND
- J3 pad 2: dac8_out_h_back -> clock_out_back
- J3 pad 3: dac8_out_f_back -> run_out_back
- J3 pad 4: dac8_out_e_back -> 1_16_out_back
- J3 pad 5: dac8_out_c_back -> var_out_back
- J3 pad 6: dac8_out_d_back -> gate_out_a_back
- J3 pad 7: dac8_out_b_back -> gate_out_b_back
- J3 pad 8: dac8_out_a_back -> gate_out_c_back
- J3 pad 9: dac4_out_c_back -> gate_out_d_back
- R12 pad 2: v_out_dac4_d -> v_out_dac4_b
- R13 pad 2: v_out_dac4_b -> v_out_dac4_d
- R16 pad 1: dac4_out_d_back -> dac4_out_b_back
- R17 pad 1: dac4_out_b_back -> dac4_out_d_back
- R20 pad 1: dac4_out_d_back -> dac4_out_b_back
- R21 pad 1: dac4_out_b_back -> dac4_out_d_back
- R25 pad 1: +3V3 -> +3.3VA
- R26 pad 2: v_out_dac8_a -> v_out_dac8_b
- R27 pad 2: v_out_dac8_b -> v_out_dac8_h
- R28 pad 2: v_out_dac8_c -> v_out_dac8_f
- R30 pad 1: dac8_out_a_back -> dac8_out_b_back
- R31 pad 1: dac8_out_b_back -> dac8_out_h_back
- R32 pad 1: dac8_out_c_back -> dac8_out_f_back
- R34 pad 1: dac8_out_a_back -> dac8_out_b_back
- R35 pad 1: dac8_out_b_back -> dac8_out_h_back
- R36 pad 1: dac8_out_c_back -> dac8_out_f_back
- R38 pad 2: v_out_dac8_e -> v_out_dac8_a
- R39 pad 2: v_out_dac8_f -> v_out_dac8_g
- R40 pad 2: v_out_dac8_g -> v_out_dac8_e
- R41 pad 2: v_out_dac8_h -> v_out_dac8_c
- R42 pad 1: dac8_out_e_back -> dac8_out_a_back
- R43 pad 1: dac8_out_f_back -> dac8_out_g_back
- R44 pad 1: dac8_out_g_back -> dac8_out_e_back
- R45 pad 1: dac8_out_h_back -> dac8_out_c_back
- R46 pad 1: dac8_out_e_back -> dac8_out_a_back
- R47 pad 1: dac8_out_f_back -> dac8_out_g_back
- R48 pad 1: dac8_out_g_back -> dac8_out_e_back
- R49 pad 1: dac8_out_h_back -> dac8_out_c_back
Routing:
- net gate_out_a_front: track 68.4 -> 5.93 mm
- net gate_out_b_front: track 65.4 -> 3.55 mm
- net v_out_dac4_a: track 12.7 -> 72.5 mm, vias 0 -> 2
- net +3.3VA: track 97.6 -> 156.7 mm, vias 6 -> 4
- net GND: track 150.9 -> 207.9 mm, vias 116 -> 140
- net v_out_dac4_d: track 15.2 -> 71.9 mm, vias 0 -> 2
- net dac8_out_b_front: track 90.8 -> 42.6 mm
- net ref_dac4: track 24.7 -> 71.0 mm, vias 0 -> 2
- net +5V: track 134.7 -> 90.3 mm, vias 0 -> 4
- net +3V3: track 295.7 -> 339.1 mm
- net v_out_dac8_a: track 8.34 -> 51.4 mm
- net dac4_out_b_front: track 74.5 -> 35.5 mm
- net ref_dac8: track 58.1 -> 96.7 mm, vias 2 -> 4
- net gate_out_b_l: track 48.2 -> 10.8 mm
- net dac8_out_c_front: track 72.8 -> 35.5 mm, vias 0 -> 1
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Other:
- board size 80.8 x 99.1 mm -> 80.8 x 109.2 mm

Commit message: Fix issues before manufacturing first prototype
The MIDI jack footprint issue (existent in the first hardware made) is also already fixed in here.
Parts:
- C11: value 4.7u -> 4u7
- C19, C29: value 3.3u -> 4u7
- R51, R52: value 140k -> 150k
- R55, R56: value 33k -> 36k
Connections:
- J9 pad 2: Net-(J9-Pad2) -> midi_in+_front
- J9 pad 4: midi_in+_front -> midi_in-_front
- J9 pad 5: midi_in-_front -> Net-(J9-Pad5)
Routing:
- net midi_in-_front: track 16.1 -> 24.0 mm
- net midi_in+_front: track 18.9 -> 12.9 mm, vias 2 -> 1

Commit message: Fix jack switches connected to ground
Connections:
- J10 pad TN: GND -> Net-(J10-PadTN)
- J11 pad TN: GND -> Net-(J11-PadTN)
- J12 pad TN: GND -> Net-(J12-PadTN)
- J13 pad TN: GND -> Net-(J13-PadTN)
- J14 pad TN: GND -> Net-(J14-PadTN)
- J16 pad TN: GND -> Net-(J16-PadTN)
- J17 pad TN: GND -> Net-(J17-PadTN)
- J18 pad TN: GND -> Net-(J18-PadTN)
- J19 pad TN: GND -> Net-(J19-PadTN)
- J20 pad TN: GND -> Net-(J20-PadTN)
- J22 pad TN: GND -> Net-(J22-PadTN)
- J23 pad TN: GND -> Net-(J23-PadTN)
- J24 pad TN: GND -> Net-(J24-PadTN)
- J25 pad TN: GND -> Net-(J25-PadTN)
- J26 pad TN: GND -> Net-(J26-PadTN)
- J27 pad TN: GND -> Net-(J27-PadTN)
- J28 pad TN: GND -> Net-(J28-PadTN)
- J29 pad TN: GND -> Net-(J29-PadTN)
- J30 pad TN: GND -> Net-(J30-PadTN)
- J31 pad TN: GND -> Net-(J31-PadTN)

Commit message: use electrolytic caps for +/-12V rails
Parts:
- C48, C49: footprint Capacitor_SMD:C_0805_2012Metric -> Capacitor_SMD:CP_Elec_5x5.3
- IC3, IC4: footprint DAC5578:SOP65P640X120-16N -> AD5328BRUZ:SOP65P640X120-16N
- moved FB1 4.09 mm to (113.3, 127.5)
- moved C54 3.87 mm to (105.7, 121.4), turned to 0 degrees
- moved C43 3.37 mm to (91.4, 122.4), turned to 270 degrees
- moved IC5 3.10 mm to (104.1, 124.7)
- moved C48 2.74 mm to (111.0, 123.4)
- moved FB2 2.70 mm to (96.0, 129.0)
- moved D3 2.58 mm to (112.3, 131.1)
- moved D4 1.97 mm to (97.5, 132.6), turned to 0 degrees
- moved L1 1.91 mm to (88.9, 122.4), turned to 270 degrees
- moved C49 1.58 mm to (97.3, 123.4)
- moved C44 1.27 mm to (85.9, 122.4)
- moved C52 1.03 mm to (102.1, 121.4)
- moved C45 0.81 mm to (83.1, 122.9), turned to 270 degrees
- moved C17 0.38 mm to (111.3, 68.1)
- moved C18 0.33 mm to (105.7, 68.6)
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Routing:
- net GND: track 207.9 -> 213.7 mm, vias 140 -> 149
- net +3.3VA: track 156.7 -> 161.4 mm
- net VEE: track 143.1 -> 147.9 mm
- net Net-(D3-Pad2): track 3.82 -> 1.93 mm
- net VCC: track 84.4 -> 83.0 mm
- net -12V: track 5.84 -> 6.97 mm
- net +5V: track 90.3 -> 89.2 mm
- net +12V: track 6.33 -> 5.36 mm
- net Net-(D4-Pad1): track 1.86 -> 2.55 mm
- net v_ref_dac4: track 19.9 -> 20.5 mm

Commit message: wire up ad5328
Parts:
- removed R25: 10k, Resistor_SMD:R_0603_1608Metric
- removed mouse-bite-2mm-slot (x4): VAL**, Panelization:mouse-bite-2mm-slot
- added J34: Expander, Connector_PinHeader_1.27mm:PinHeader_2x03_P1.27mm_Vertical, B.Cu at (96.9, 78.2)
- added J35: SPI3 Testpoint, Connector_PinHeader_2.54mm:PinHeader_1x03_P2.54mm_Vertical, B.Cu at (106.8, 72.3)
- C29: value 4u7 -> 10u
- IC4: value DAC5578SPWR -> AD5328BRUZ
- J32: value Conn_02x05_Odd_Even -> Debug
- moved C32 10.5 mm to (101.2, 81.1)
- moved C33 10.5 mm to (99.7, 81.1)
- moved R23 10.5 mm to (98.2, 81.1)
- moved R24 10.5 mm to (96.6, 81.1)
- moved C29 8.95 mm to (100.2, 75.6), turned to 90 degrees
- moved C27 8.04 mm to (101.7, 75.6), turned to 270 degrees
- moved IC4 3.40 mm to (106.6, 77.4), turned to 0 degrees
Connections:
- IC4 pad 10: v_out_dac8_h -> v_out_dac8_e
- IC4 pad 12: v_out_dac8_d -> v_out_dac8_g
- IC4 pad 13: v_out_dac8_b -> v_out_dac8_h
- IC4 pad 15: i2c3_sda -> spi3_mosi
- IC4 pad 16: i2c3_scl -> spi3_sck
- IC4 pad 2: GND -> spi3_nss
- IC4 pad 5: v_out_dac8_c -> v_out_dac8_b
- IC4 pad 6: v_out_dac8_e -> v_out_dac8_c
- IC4 pad 7: v_out_dac8_g -> v_out_dac8_d
- IC4 pad 9: Net-(IC4-Pad9) -> v_ref_dac4
- J4 pad 1: dac8_out_c_back -> dac8_out_g_back
- J4 pad 2: dac8_out_e_back -> dac8_out_f_back
- J4 pad 3: dac8_out_f_back -> dac8_out_b_back
- J4 pad 4: dac8_out_d_back -> dac8_out_c_back
- J4 pad 5: dac8_out_b_back -> dac8_out_h_back
- J4 pad 6: dac8_out_h_back -> dac8_out_e_back
- J4 pad 7: dac8_out_g_back -> dac8_out_a_back
- J4 pad 8: dac8_out_a_back -> dac8_out_d_back
- J8 pad 1: dac8_out_c_front -> dac8_out_g_front
- J8 pad 2: dac8_out_e_front -> dac8_out_f_front
- J8 pad 3: dac8_out_f_front -> dac8_out_b_front
- J8 pad 4: dac8_out_d_front -> dac8_out_c_front
- J8 pad 5: dac8_out_b_front -> dac8_out_h_front
- J8 pad 6: dac8_out_h_front -> dac8_out_e_front
- J8 pad 7: dac8_out_g_front -> dac8_out_a_front
- J8 pad 8: dac8_out_a_front -> dac8_out_d_front
- R26 pad 2: v_out_dac8_b -> v_out_dac8_d
- R27 pad 2: v_out_dac8_h -> v_out_dac8_a
- R28 pad 2: v_out_dac8_f -> v_out_dac8_b
- R29 pad 2: v_out_dac8_d -> v_out_dac8_c
- R30 pad 1: dac8_out_b_back -> dac8_out_d_back
- R31 pad 1: dac8_out_h_back -> dac8_out_a_back
- R32 pad 1: dac8_out_f_back -> dac8_out_b_back
- R33 pad 1: dac8_out_d_back -> dac8_out_c_back
- R34 pad 1: dac8_out_b_back -> dac8_out_d_back
- R35 pad 1: dac8_out_h_back -> dac8_out_a_back
- R36 pad 1: dac8_out_f_back -> dac8_out_b_back
- R37 pad 1: dac8_out_d_back -> dac8_out_c_back
- R38 pad 2: v_out_dac8_a -> v_out_dac8_e
- R39 pad 2: v_out_dac8_g -> v_out_dac8_h
- R40 pad 2: v_out_dac8_e -> v_out_dac8_g
- R41 pad 2: v_out_dac8_c -> v_out_dac8_f
- R42 pad 1: dac8_out_a_back -> dac8_out_e_back
- R43 pad 1: dac8_out_g_back -> dac8_out_h_back
- R44 pad 1: dac8_out_e_back -> dac8_out_g_back
- R45 pad 1: dac8_out_c_back -> dac8_out_f_back
- R46 pad 1: dac8_out_a_back -> dac8_out_e_back
- R47 pad 1: dac8_out_g_back -> dac8_out_h_back
- R48 pad 1: dac8_out_e_back -> dac8_out_g_back
- R49 pad 1: dac8_out_c_back -> dac8_out_f_back
- U3 pad 50: Net-(U3-Pad50) -> spi3_nss
- U3 pad 51: Net-(U3-Pad51) -> spi3_sck
- U3 pad 53: Net-(U3-Pad53) -> spi3_mosi
Routing:
- net dac8_out_a_front: track 40.2 -> 85.7 mm
- net v_out_dac8_g: track 68.3 -> 43.1 mm
- net spi3_mosi: track 0.00 -> 24.7 mm, vias 0 -> 1
- net v_ref_dac4: track 20.5 -> 43.0 mm, vias 0 -> 3
- net spi3_sck: track 0.00 -> 20.3 mm, vias 0 -> 1
- net spi3_nss: track 0.00 -> 19.5 mm, vias 0 -> 1
- net v_out_dac8_c: track 39.1 -> 20.5 mm
- net dac8_out_c_back: track 21.3 -> 37.2 mm
- net dac8_out_h_back: track 25.9 -> 10.2 mm
- net dac8_out_e_back: track 9.20 -> 24.2 mm
- net ref_dac8: track 96.7 -> 84.2 mm
- net dac8_out_b_back: track 36.4 -> 24.1 mm
- net dac8_out_c_front: track 35.5 -> 45.9 mm, vias 1 -> 0
- net +3V3: track 339.3 -> 349.5 mm
- net v_out_dac8_b: track 36.6 -> 27.3 mm
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
Commit message: make back compatible with old front
Connections:
- J4 pad 1: dac8_out_g_back -> dac8_out_c_back
- J4 pad 2: dac8_out_f_back -> dac8_out_e_back
- J4 pad 3: dac8_out_b_back -> dac8_out_f_back
- J4 pad 4: dac8_out_c_back -> dac8_out_d_back
- J4 pad 5: dac8_out_h_back -> dac8_out_b_back
- J4 pad 6: dac8_out_e_back -> dac8_out_h_back
- J4 pad 7: dac8_out_a_back -> dac8_out_g_back
- J4 pad 8: dac8_out_d_back -> dac8_out_a_back
- J8 pad 1: dac8_out_g_front -> dac8_out_c_front
- J8 pad 2: dac8_out_f_front -> dac8_out_e_front
- J8 pad 3: dac8_out_b_front -> dac8_out_f_front
- J8 pad 4: dac8_out_c_front -> dac8_out_d_front
- J8 pad 5: dac8_out_h_front -> dac8_out_b_front
- J8 pad 6: dac8_out_e_front -> dac8_out_h_front
- J8 pad 7: dac8_out_a_front -> dac8_out_g_front
- J8 pad 8: dac8_out_d_front -> dac8_out_a_front
Routing:
- net dac8_out_a_front: track 85.7 -> 38.9 mm
- net dac8_out_b_back: track 24.1 -> 41.2 mm
- net dac8_out_e_front: track 4.96 -> 20.6 mm
- net dac8_out_b_front: track 39.1 -> 52.3 mm
- net dac8_out_h_front: track 17.9 -> 26.3 mm
- net dac8_out_g_back: track 10.3 -> 18.5 mm, vias 1 -> 2
- net dac8_out_d_back: track 37.7 -> 44.1 mm
- net dac8_out_e_back: track 24.2 -> 30.5 mm
- net dac8_out_g_front: track 12.9 -> 7.50 mm
- net dac8_out_f_front: track 4.58 -> 7.12 mm
- net dac8_out_d_front: track 38.2 -> 36.3 mm
- net dac8_out_h_back: track 10.2 -> 9.08 mm
- net dac8_out_a_back: track 26.9 -> 26.1 mm
- net GND: track 217.5 -> 218.3 mm, vias 159 -> 156
- net dac8_out_c_back: track 37.2 -> 36.4 mm
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Other:
- outline, holes or cut-outs redrawn
