File: hardware/cv_input.sch (KiCad schematic (older format))
At the start: 14 parts, among them U10 MCP6002-xMS

Commit message: Fix issues before manufacturing first prototype
The MIDI jack footprint issue (existent in the first hardware made) is also already fixed in here.
Parts:
- D5, D6: LCSC (none) -> C210791; LCSC Part # (none) -> C210791
- R51, R52: value 140k -> 150k; LCSC (none) -> C22807; LCSC Part # (none) -> C22807
- R55, R56: value 33k -> 36k; LCSC C4216 -> C23147; LCSC Part # C4216 -> C23147
Changed lines of the file:
@@
 AR Path="/61005BD4/612EE3A1/5FCFEC8F" Ref="R55"  Part="1"
 F 0 "R55" V 3993 2750 50  0000 C CNN
-F 1 "33k" V 4084 2750 50  0000 C CNN
+F 1 "36k" V 4084 2750 50  0000 C CNN
 F 2 "Resistor_SMD:R_0603_1608Metric" V 4130 2750 50  0001 C CNN
 F 3 "~" H 4200 2750 50  0001 C CNN
-F 4 "C4216" H 4200 2750 50  0001 C CNN "LCSC Part #"
-F 5 "C4216" H 4200 2750 50  0001 C CNN "LCSC"
+F 4 "C23147" H 4200 2750 50  0001 C CNN "LCSC Part #"
+F 5 "C23147" H 4200 2750 50  0001 C CNN "LCSC"
 	1    4200 2750
 	0    1    1    0
@@
 AR Path="/61005BD4/612EE3A1/5FCFEC9C" Ref="R51"  Part="1"
 F 0 "R51" V 2643 2250 50  0000 C CNN
-F 1 "140k" V 2734 2250 50  0000 C CNN
+F 1 "150k" V 2734 2250 50  0000 C CNN
 F 2 "Resistor_SMD:R_0603_1608Metric" V 2780 2250 50  0001 C CNN
 F 3 "~" H 2850 2250 50  0001 C CNN
+F 4 "C22807" H 2850 2250 50  0001 C CNN "LCSC Part #"
+F 5 "C22807" H 2850 2250 50  0001 C CNN "LCSC"
 	1    2850 2250
 	0    1    1    0
@@
 F 2 "Diode_SMD:D_0603_1608Metric" H 2500 2500 50  0001 C CNN
 F 3 "https://product.tdk.com/info/en/documents/data_sheet/75/ds/High_speed_series.pdf" H 2500 2500 50  0001 C CNN
+F 4 "C210791" H 2500 2500 50  0001 C CNN "LCSC Part #"
+F 5 "C210791" H 2500 2500 50  0001 C CNN "LCSC"
 	1    2500 2500
 	0    1    1    0
@@
 AR Path="/61005BD4/612EE3A1/5FE5D6A7" Ref="R56"  Part="1"
 F 0 "R56" V 3993 5700 50  0000 C CNN
-F 1 "33k" V 4084 5700 50  0000 C CNN
+F 1 "36k" V 4084 5700 50  0000 C CNN
 F 2 "Resistor_SMD:R_0603_1608Metric" V 4130 5700 50  0001 C CNN
 F 3 "~" H 4200 5700 50  0001 C CNN
-F 4 "C4216" H 4200 5700 50  0001 C CNN "LCSC Part #"
-F 5 "C4216" H 4200 5700 50  0001 C CNN "LCSC"
+F 4 "C23147" H 4200 5700 50  0001 C CNN "LCSC Part #"
+F 5 "C23147" H 4200 5700 50  0001 C CNN "LCSC"
 	1    4200 5700
 	0    1    1    0
@@
 AR Path="/61005BD4/612EE3A1/5FE5D6AF" Ref="R52"  Part="1"
 F 0 "R52" V 2643 5200 50  0000 C CNN
-F 1 "140k" V 2734 5200 50  0000 C CNN
+F 1 "150k" V 2734 5200 50  0000 C CNN
 F 2 "Resistor_SMD:R_0603_1608Metric" V 2780 5200 50  0001 C CNN
 F 3 "~" H 2850 5200 50  0001 C CNN
+F 4 "C22807" H 2850 5200 50  0001 C CNN "LCSC Part #"
+F 5 "C22807" H 2850 5200 50  0001 C CNN "LCSC"
 	1    2850 5200
 	0    1    1    0
@@
 F 2 "Diode_SMD:D_0603_1608Metric" H 2500 5450 50  0001 C CNN
 F 3 "https://product.tdk.com/info/en/documents/data_sheet/75/ds/High_speed_series.pdf" H 2500 5450 50  0001 C CNN
+F 4 "C210791" H 2500 5450 50  0001 C CNN "LCSC Part #"
+F 5 "C210791" H 2500 5450 50  0001 C CNN "LCSC"
 	1    2500 5450
 	0    1    1    0
