File: hardware/dac4.sch (KiCad schematic (older format))
At the start: 5 parts

Commit message: Add amplifier circuits for DACs
Parts:
- added C? (x2): 100n, symbol Device:C
- added C? (x4): 22p, symbol Device:C
- added R?: 36k, symbol Device:R
- added R? (x5): 33k, symbol Device:R
- added R? (x4): 1k, symbol Device:R
- added R? (x4): 180k, symbol Device:R
- added U? (x5): OPA4172, Package_SO:TSSOP-14_4.4x5mm_P0.65mm, symbol Amplifier_Operational:TL074
Connections:
- net GND: now also C?.1, C?.1, R?.1
- net v_out_dac4_a: now reaches IC?.1 (VOUTA)
- net v_out_dac4_a: now also R?.2
- net v_out_dac4_b: now reaches IC?.2 (VOUTB)
- net v_out_dac4_b: now also R?.2
- net v_out_dac4_c: now reaches IC?.7 (VOUTC)
- net v_out_dac4_c: now also R?.2
- net v_out_dac4_d: now reaches IC?.8 (VOUTD)
- net v_out_dac4_d: now also R?.2
- net v_ref_dac renamed v_ref
- net v_ref: now also R?.1
- new net: C?.1, R?.1, R?.2, U?.2 (-)
- new net: C?.2, R?.2, U?.1
- new net: C?.1, R?.1, R?.2, U?.6 (-)
- new net: C?.2, R?.2, U?.7
- new net: C?.1, R?.1, R?.2, U?.9 (-)
- new net: C?.2, R?.2, U?.8
- new net: C?.1, R?.1, R?.2, U?.13 (-)
- new net: C?.2, R?.2, U?.14
- new net +12V: C?.2, U?.4 (V+)
- new net -12V: C?.2, U?.11 (V-)
- new net note_out_a: R?.1, R?.1
- new net note_out_b: R?.1, R?.1
- new net note_out_c: R?.1, R?.1
- new net note_out_d: R?.1, R?.1
- new net ref_dac4: R?.2, R?.2, U?.10 (+), U?.12 (+), U?.3 (+), U?.5 (+)
Other:
- note added: "-5.2V to 8.4V"
- moved on the sheet: C?, IC?

Commit message: First preliminary board design
Parts:
- C17, C18, C19, C20, C21, C22, C23, C24, C25, C26: renamed from C?; footprint (none) -> Capacitor_SMD:C_0603_1608Metric
- R10, R11, R12, R13, R14, R15, R16, R17, R18, R19, R20, R21, R22, R9: renamed from R?; footprint (none) -> Resistor_SMD:R_0603_1608Metric
- gave numbers to parts that had none: 2
Connections:
- net +12V renamed VCC
- net -12V renamed VEE
- net note_out_a renamed dac4_out_a
- net note_out_b renamed dac4_out_b
- net note_out_c renamed dac4_out_c
- net note_out_d renamed dac4_out_d
- net v_ref renamed v_ref_dac4
Other:
- moved on the sheet: C21, C22

Commit message: Layed out stretched design
Connections:
- net dac4_out_b: now also R16.1, R20.1; no longer R17.1, R21.1
- net dac4_out_d: now also R17.1, R21.1; no longer R16.1, R20.1
- net v_out_dac4_b: now also R12.2; no longer R13.2
- net v_out_dac4_d: now also R13.2; no longer R12.2
Changed lines of the file:
@@
 $EndDescr
 $Comp
-L power:GND #PWR0113
+L power:GND #PWR0115
 U 1 1 60A46579
 P 4450 5150
-F 0 "#PWR0113" H 4450 4900 50  0001 C CNN
+F 0 "#PWR0115" H 4450 4900 50  0001 C CNN
 F 1 "GND" H 4455 4977 50  0000 C CNN
 F 2 "" H 4450 5150 50  0001 C CNN
@@
 $EndComp
 $Comp
-L power:+3.3VA #PWR0106
+L power:+3.3VA #PWR0108
 U 1 1 60A46C2F
 P 2250 1350
-F 0 "#PWR0106" H 2250 1200 50  0001 C CNN
+F 0 "#PWR0108" H 2250 1200 50  0001 C CNN
 F 1 "+3.3VA" H 2265 1523 50  0000 C CNN
 F 2 "" H 2250 1350 50  0001 C CNN
@@
 $EndComp
 $Comp
-L power:+3.3V #PWR0101
+L power:+3.3V #PWR0103
 U 1 1 60A4736E
 P 1450 1350
-F 0 "#PWR0101" H 1450 1200 50  0001 C CNN
+F 0 "#PWR0103" H 1450 1200 50  0001 C CNN
 F 1 "+3.3V" H 1465 1523 50  0000 C CNN
 F 2 "" H 1450 1350 50  0001 C CNN
@@
 $EndComp
 $Comp
-L power:GND #PWR0107
+L power:GND #PWR0109
 U 1 1 60A48509
 P 2250 1850
-F 0 "#PWR0107" H 2250 1600 50  0001 C CNN
+F 0 "#PWR0109" H 2250 1600 50  0001 C CNN
 F 1 "GND" H 2255 1677 50  0000 C CNN
 F 2 "" H 2250 1850 50  0001 C CNN
@@
 Connection ~ 2250 1850
 $Comp
-L power:+3.3VA #PWR0103
+L power:+3.3VA #PWR0105
 U 1 1 60A4E5A0
 P 1950 5650
-F 0 "#PWR0103" H 1950 5500 50  0001 C CNN
+F 0 "#PWR0105" H 1950 5500 50  0001 C CNN
 F 1 "+3.3VA" V 1965 5777 50  0000 L CNN
 F 2 "" H 1950 5650 50  0001 C CNN
@@
 	1950 5650 2450 5650
 $Comp
-L power:GND #PWR0105
+L power:GND #PWR0107
 U 1 1 60A48919
 P 2150 5750
-F 0 "#PWR0105" H 2150 5500 50  0001 C CNN
+F 0 "#PWR0107" H 2150 5500 50  0001 C CNN
 F 1 "GND" V 2155 5622 50  0000 R CNN
 F 2 "" H 2150 5750 50  0001 C CNN
@@
 v_ref_dac4
 $Comp
-L power:GND #PWR0108
+L power:GND #PWR0110
 U 1 1 60A528A6
 P 3000 1850
-F 0 "#PWR0108" H 3000 1600 50  0001 C CNN
+F 0 "#PWR0110" H 3000 1600 50  0001 C CNN
 F 1 "GND" H 3005 1677 50  0000 C CNN
 F 2 "" H 3000 1850 50  0001 C CNN
@@
 	4450 5350 4450 5150
 $Comp
-L power:+3.3V #PWR0116
+L power:+3.3V #PWR0118
 U 1 1 60A5711A
 P 4650 5750
-F 0 "#PWR0116" H 4650 5600 50  0001 C CNN
+F 0 "#PWR0118" H 4650 5600 50  0001 C CNN
 F 1 "+3.3V" V 4665 5878 50  0000 L CNN
 F 2 "" H 4650 5750 50  0001 C CNN
@@
 	1450 1450 1450 1350
 $Comp
-L power:GND #PWR0102
+L power:GND #PWR0104
 U 1 1 60A5AAE5
 P 1450 1850
-F 0 "#PWR0102" H 1450 1600 50  0001 C CNN
+F 0 "#PWR0104" H 1450 1600 50  0001 C CNN
 F 1 "GND" H 1455 1677 50  0000 C CNN
 F 2 "" H 1450 1850 50  0001 C CNN
@@
 $EndComp
 $Comp
-L power:GND #PWR0104
+L power:GND #PWR0106
 U 1 1 60B20046
 P 2050 4250
-F 0 "#PWR0104" H 2050 4000 50  0001 C CNN
+F 0 "#PWR0106" H 2050 4000 50  0001 C CNN
 F 1 "GND" H 2055 4077 50  0000 C CNN
 F 2 "" H 2050 4250 50  0001 C CNN
@@
 	3950 1450 3950 1350
 $Comp
-L power:GND #PWR0110
+L power:GND #PWR0112
 U 1 1 60B61C61
 P 3950 1850
-F 0 "#PWR0110" H 3950 1600 50  0001 C CNN
+F 0 "#PWR0112" H 3950 1600 50  0001 C CNN
 F 1 "GND" H 3955 1677 50  0000 C CNN
 F 2 "" H 3950 1850 50  0001 C CNN
@@
 	4600 1450 4600 1350
 $Comp
-L power:GND #PWR0115
+L power:GND #PWR0117
 U 1 1 60B68A44
 P 4600 1850
-F 0 "#PWR0115" H 4600 1600 50  0001 C CNN
+F 0 "#PWR0117" H 4600 1600 50  0001 C CNN
 F 1 "GND" H 4605 1677 50  0000 C CNN
 F 2 "" H 4600 1850 50  0001 C CNN
@@
 ref_dac4
 Text GLabel 6550 2500 0    50   Input ~ 0
-v_out_dac4_b
+v_out_dac4_d
 Text Notes 9350 2300 0    50   ~ 0
 -5.2V to 8.4V
@@
 ref_dac4
 Text GLabel 6500 5300 0    50   Input ~ 0
-v_out_dac4_d
+v_out_dac4_b
 Text Notes 9300 5100 0    50   ~ 0
 -5.2V to 8.4V
@@
 dac4_out_a
 Text HLabel 9400 2400 2    50   Output ~ 0
-dac4_out_b
+dac4_out_d
 Text HLabel 9400 3800 2    50   Output ~ 0
 dac4_out_c
 Text HLabel 9350 5200 2    50   Output ~ 0
-dac4_out_d
+dac4_out_b
 Text HLabel 3350 1450 2    50   Output ~ 0
 v_ref
@@
 Connection ~ 3000 1450
 $Comp
-L power:VCC #PWR0109
+L power:VCC #PWR0111
 U 1 1 611B727E
 P 3950 1350
-F 0 "#PWR0109" H 3950 1200 50  0001 C CNN
+F 0 "#PWR0111" H 3950 1200 50  0001 C CNN
 F 1 "VCC" H 3965 1523 50  0000 C CNN
 F 2 "" H 3950 1350 50  0001 C CNN
@@
 $EndComp
 $Comp
-L power:VEE #PWR0111
+L power:VEE #PWR0116
 U 1 1 611B8584
 P 4600 1350
-F 0 "#PWR0111" H 4600 1200 50  0001 C CNN
+F 0 "#PWR0116" H 4600 1200 50  0001 C CNN
 F 1 "VEE" H 4615 1523 50  0000 C CNN
 F 2 "" H 4600 1350 50  0001 C CNN
@@
 $EndComp
 $Comp
-L power:VCC #PWR0112
+L power:VCC #PWR0113
 U 1 1 611B9B4A
 P 4050 3400
-F 0 "#PWR0112" H 4050 3250 50  0001 C CNN
+F 0 "#PWR0113" H 4050 3250 50  0001 C CNN
 F 1 "VCC" H 4065 3573 50  0000 C CNN
 F 2 "" H 4050 3400 50  0001 C CNN

Commit message: Fix issues before manufacturing first prototype
The MIDI jack footprint issue (existent in the first hardware made) is also already fixed in here.
Parts:
- C17, C18, C21, C22: LCSC (none) -> C14663; LCSC Part # (none) -> C14663
- C19: value 3.3u -> 4u7; LCSC (none) -> C19666; LCSC Part # (none) -> C19666
- C20: LCSC (none) -> C21120; LCSC Part # (none) -> C21120
- C23, C24, C25, C26: LCSC (none) -> C1653; LCSC Part # (none) -> C1653
- IC3: LCSC (none) -> C1554750; LCSC Part # (none) -> C1554750
- R10: LCSC (none) -> C23147; LCSC Part # (none) -> C23147
- R11, R12, R13, R14, R9: LCSC (none) -> C4216; LCSC Part # (none) -> C4216
- R15, R16, R17, R18: LCSC (none) -> C22827; LCSC Part # (none) -> C22827
- R19, R20, R21, R22: LCSC (none) -> C21190; LCSC Part # (none) -> C21190
Changed lines of the file:
@@
 P 2450 1600
 F 0 "C19" H 2565 1646 50  0000 L CNN
-F 1 "3.3u" H 2565 1555 50  0000 L CNN
+F 1 "4u7" H 2565 1555 50  0000 L CNN
 F 2 "Capacitor_SMD:C_0603_1608Metric" H 2488 1450 50  0001 C CNN
 F 3 "~" H 2450 1600 50  0001 C CNN
+F 4 "C19666" H 2450 1600 50  0001 C CNN "LCSC Part #"
+F 5 "C19666" H 2450 1600 50  0001 C CNN "LCSC"
 	1    2450 1600
 	1    0    0    -1
@@
 F 2 "Capacitor_SMD:C_0603_1608Metric" H 2088 1450 50  0001 C CNN
 F 3 "~" H 2050 1600 50  0001 C CNN
+F 4 "C14663" H 2050 1600 50  0001 C CNN "LCSC Part #"
+F 5 "C14663" H 2050 1600 50  0001 C CNN "LCSC"
 	1    2050 1600
 	-1   0    0    1
@@
 F 2 "Capacitor_SMD:C_0603_1608Metric" H 3038 1450 50  0001 C CNN
 F 3 "~" H 3000 1600 50  0001 C CNN
+F 4 "C21120" H 3000 1600 50  0001 C CNN "LCSC Part #"
+F 5 "C21120" H 3000 1600 50  0001 C CNN "LCSC"
 	1    3000 1600
 	-1   0    0    1
@@
 F 2 "Capacitor_SMD:C_0603_1608Metric" H 1488 1450 50  0001 C CNN
 F 3 "~" H 1450 1600 50  0001 C CNN
+F 4 "C14663" H 1450 1600 50  0001 C CNN "LCSC Part #"
+F 5 "C14663" H 1450 1600 50  0001 C CNN "LCSC"
 	1    1450 1600
 	-1   0    0    1
@@
 F 10 "DAC8564IAPW" H 4100 4650 50  0001 L CNN "Arrow Part Number"
 F 11 "https://www.arrow.com/en/products/dac8564iapw/texas-instruments" H 4100 4550 50  0001 L CNN "Arrow Price/Stock"
+F 12 "C1554750" H 2450 5350 50  0001 C CNN "LCSC Part #"
+F 13 "C1554750" H 2450 5350 50  0001 C CNN "LCSC"
 	1    2450 5350
 	1    0    0    -1
@@
 F 2 "Resistor_SMD:R_0603_1608Metric" V 6980 1100 50  0001 C CNN
 F 3 "~" H 7050 1100 50  0001 C CNN
+F 4 "C4216" H 7050 1100 50  0001 C CNN "LCSC Part #"
+F 5 "C4216" H 7050 1100 50  0001 C CNN "LCSC"
 	1    7050 1100
 	0    1    1    0
@@
 F 2 "Resistor_SMD:R_0603_1608Metric" V 8780 1000 50  0001 C CNN
 F 3 "~" H 8850 1000 50  0001 C CNN
+F 4 "C21190" H 8850 1000 50  0001 C CNN "LCSC Part #"
+F 5 "C21190" H 8850 1000 50  0001 C CNN "LCSC"
 	1    8850 1000
 	0    1    1    0
@@
 F 2 "Resistor_SMD:R_0603_1608Metric" V 8130 1900 50  0001 C CNN
 F 3 "~" H 8200 1900 50  0001 C CNN
+F 4 "C22827" H 8200 1900 50  0001 C CNN "LCSC Part #"
+F 5 "C22827" H 8200 1900 50  0001 C CNN "LCSC"
 	1    8200 1900
 	0    1    1    0
@@
 F 2 "Resistor_SMD:R_0603_1608Metric" V 1980 4000 50  0001 C CNN
 F 3 "~" H 2050 4000 50  0001 C CNN
+F 4 "C23147" H 2050 4000 50  0001 C CNN "LCSC Part #"
+F 5 "C23147" H 2050 4000 50  0001 C CNN "LCSC"
 	1    2050 4000
 	-1   0    0    1
@@
 F 2 "Resistor_SMD:R_0603_1608Metric" V 1980 3400 50  0001 C CNN
 F 3 "~" H 2050 3400 50  0001 C CNN
+F 4 "C4216" H 2050 3400 50  0001 C CNN "LCSC Part #"
+F 5 "C4216" H 2050 3400 50  0001 C CNN "LCSC"
 	1    2050 3400
 	1    0    0    -1
@@
 F 2 "Capacitor_SMD:C_0603_1608Metric" H 3988 1450 50  0001 C CNN
 F 3 "~" H 3950 1600 50  0001 C CNN
+F 4 "C14663" H 3950 1600 50  0001 C CNN "LCSC Part #"
+F 5 "C14663" H 3950 1600 50  0001 C CNN "LCSC"
 	1    3950 1600
 	-1   0    0    1
@@
 F 2 "Capacitor_SMD:C_0603_1608Metric" H 4638 1450 50  0001 C CNN
 F 3 "~" H 4600 1600 50  0001 C CNN
+F 4 "C14663" H 4600 1600 50  0001 C CNN "LCSC Part #"
+F 5 "C14663" H 4600 1600 50  0001 C CNN "LCSC"
 	1    4600 1600
 	-1   0    0    1
@@
 F 2 "Capacitor_SMD:C_0603_1608Metric" H 7988 1350 50  0001 C CNN
 F 3 "~" H 7950 1500 50  0001 C CNN
+F 4 "C1653" H 7950 1500 50  0001 C CNN "LCSC Part #"
+F 5 "C1653" H 7950 1500 50  0001 C CNN "LCSC"
 	1    7950 1500
 	0    -1   -1   0
@@
 F 2 "Resistor_SMD:R_0603_1608Metric" V 7030 2500 50  0001 C CNN
 F 3 "~" H 7100 2500 50  0001 C CNN
+F 4 "C4216" H 7100 2500 50  0001 C CNN "LCSC Part #"
+F 5 "C4216" H 7100 2500 50  0001 C CNN "LCSC"
 	1    7100 2500
 	0    1    1    0
@@
 F 2 "Resistor_SMD:R_0603_1608Metric" V 8830 2400 50  0001 C CNN
 F 3 "~" H 8900 2400 50  0001 C CNN
+F 4 "C21190" H 8900 2400 50  0001 C CNN "LCSC Part #"
+F 5 "C21190" H 8900 2400 50  0001 C CNN "LCSC"
 	1    8900 2400
 	0    1    1    0
@@
 F 2 "Resistor_SMD:R_0603_1608Metric" V 8180 3300 50  0001 C CNN
 F 3 "~" H 8250 3300 50  0001 C CNN
+F 4 "C22827" H 8250 3300 50  0001 C CNN "LCSC Part #"
+F 5 "C22827" H 8250 3300 50  0001 C CNN "LCSC"
 	1    8250 3300
 	0    1    1    0
@@
 F 2 "Capacitor_SMD:C_0603_1608Metric" H 8038 2750 50  0001 C CNN
 F 3 "~" H 8000 2900 50  0001 C CNN
+F 4 "C1653" H 8000 2900 50  0001 C CNN "LCSC Part #"
+F 5 "C1653" H 8000 2900 50  0001 C CNN "LCSC"
 	1    8000 2900
 	0    -1   -1   0
@@
 F 2 "Resistor_SMD:R_0603_1608Metric" V 7030 3900 50  0001 C CNN
 F 3 "~" H 7100 3900 50  0001 C CNN
+F 4 "C4216" H 7100 3900 50  0001 C CNN "LCSC Part #"
+F 5 "C4216" H 7100 3900 50  0001 C CNN "LCSC"
 	1    7100 3900
 	0    1    1    0
@@
 F 2 "Resistor_SMD:R_0603_1608Metric" V 8830 3800 50  0001 C CNN
 F 3 "~" H 8900 3800 50  0001 C CNN
+F 4 "C21190" H 8900 3800 50  0001 C CNN "LCSC Part #"
+F 5 "C21190" H 8900 3800 50  0001 C CNN "LCSC"
 	1    8900 3800
 	0    1    1    0
@@
 F 2 "Resistor_SMD:R_0603_1608Metric" V 8180 4700 50  0001 C CNN
 F 3 "~" H 8250 4700 50  0001 C CNN
+F 4 "C22827" H 8250 4700 50  0001 C CNN "LCSC Part #"
+F 5 "C22827" H 8250 4700 50  0001 C CNN "LCSC"
 	1    8250 4700
 	0    1    1    0
@@
 F 2 "Capacitor_SMD:C_0603_1608Metric" H 8038 4150 50  0001 C CNN
 F 3 "~" H 8000 4300 50  0001 C CNN
+F 4 "C1653" H 8000 4300 50  0001 C CNN "LCSC Part #"
+F 5 "C1653" H 8000 4300 50  0001 C CNN "LCSC"
 	1    8000 4300
 	0    -1   -1   0
@@
 F 2 "Resistor_SMD:R_0603_1608Metric" V 6980 5300 50  0001 C CNN
 F 3 "~" H 7050 5300 50  0001 C CNN
+F 4 "C4216" H 7050 5300 50  0001 C CNN "LCSC Part #"
+F 5 "C4216" H 7050 5300 50  0001 C CNN "LCSC"
 	1    7050 5300
 	0    1    1    0
@@
 F 2 "Resistor_SMD:R_0603_1608Metric" V 8780 5200 50  0001 C CNN
 F 3 "~" H 8850 5200 50  0001 C CNN
+F 4 "C21190" H 8850 5200 50  0001 C CNN "LCSC Part #"
+F 5 "C21190" H 8850 5200 50  0001 C CNN "LCSC"
 	1    8850 5200
 	0    1    1    0
@@
 F 2 "Resistor_SMD:R_0603_1608Metric" V 8130 6100 50  0001 C CNN
 F 3 "~" H 8200 6100 50  0001 C CNN
+F 4 "C22827" H 8200 6100 50  0001 C CNN "LCSC Part #"
+F 5 "C22827" H 8200 6100 50  0001 C CNN "LCSC"
 	1    8200 6100
 	0    1    1    0
@@
 F 2 "Capacitor_SMD:C_0603_1608Metric" H 7988 5550 50  0001 C CNN
 F 3 "~" H 7950 5700 50  0001 C CNN
+F 4 "C1653" H 7950 5700 50  0001 C CNN "LCSC Part #"
+F 5 "C1653" H 7950 5700 50  0001 C CNN "LCSC"
 	1    7950 5700
 	0    -1   -1   0
