File: hardware/dac8.sch (KiCad schematic (older format))
At the start: 4 parts

Commit message: Add amplifier circuits for DACs
Parts:
- removed C?: 3.3u, symbol Device:C
- removed C?: 100n, symbol Device:C
- added C? (x8): 10p, symbol Device:C
- added C?: 3.3u, symbol Device:C
- added C? (x5): 100n, symbol Device:C
- added R? (x8): 150k, symbol Device:R
- added R? (x8): 36k, symbol Device:R
- added R? (x8): 1k, symbol Device:R
- added R?: 22k, symbol Device:R
- added R?: 33k, symbol Device:R
- added U? (x9): TL074, Package_SO:TSSOP-14_4.4x5mm_P0.65mm, symbol Amplifier_Operational:TL074
- added U?: TL074, symbol Amplifier_Operational:TL074
Connections:
- net labels added: +12V, -12V, mod_out_a, mod_out_b, mod_out_c, mod_out_d, mod_out_e, mod_out_f, mod_out_g, mod_out_h, ref_dac8, v_out_dac8_a, v_out_dac8_b, v_out_dac8_c, v_out_dac8_d, v_out_dac8_e, v_out_dac8_f, v_out_dac8_g, v_out_dac8_h, v_ref
- wire segments 16 -> 149
Other:
- note added: "-5.2V to 5.2V"
- moved on the sheet: R?

Commit message: First preliminary board design
Parts:
- added C32: 1u, Capacitor_SMD:C_0603_1608Metric, symbol Device:C
- added C33: 100n, Capacitor_SMD:C_0603_1608Metric, symbol Device:C
- C27, C28, C29, C30, C31, C34, C35, C36, C37, C38, C39, C40, C41, C42: renamed from C?; footprint (none) -> Capacitor_SMD:C_0603_1608Metric
- R23, R24, R25, R26, R27, R28, R29, R30, R31, R32, R33, R34, R35, R36, R37, R38, R39, R40, R41, R42, R43, R44, R45, R46, R47, R48, R49: renamed from R?; footprint (none) -> Resistor_SMD:R_0603_1608Metric
- U6: renamed from U?; footprint (none) -> Package_SO:TSSOP-14_4.4x5mm_P0.65mm
- gave numbers to parts that had none: 3
Connections:
- net labels added: VCC, VEE, dac8_out_a, dac8_out_b, dac8_out_c, dac8_out_d, dac8_out_e, dac8_out_f, dac8_out_g, dac8_out_h, v_ref_dac8
- net labels removed: +12V, -12V, mod_out_a, mod_out_b, mod_out_c, mod_out_d, mod_out_e, mod_out_f, mod_out_g, mod_out_h, v_ref_dac
- wire segments 149 -> 154
Other:
- moved on the sheet: C27, C29

Commit message: Layed out stretched design
Connections:
- net labels removed: +3.3V
Changed lines of the file:
@@
 $EndComp
 $Comp
-L power:+3.3VA #PWR0122
+L power:+3.3VA #PWR0124
 U 1 1 60A68DBC
 P 1300 6450
-F 0 "#PWR0122" H 1300 6300 50  0001 C CNN
+F 0 "#PWR0124" H 1300 6300 50  0001 C CNN
 F 1 "+3.3VA" V 1315 6577 50  0000 L CNN
 F 2 "" H 1300 6450 50  0001 C CNN
@@
 AR Path="/60A48B70/60A68DC3" Ref="#PWR?"  Part="1"
 AR Path="/60A5BF82/60A68DC3" Ref="#PWR?"  Part="1"
-AR Path="/61005BD4/60A5BF82/60A68DC3" Ref="#PWR0125"  Part="1"
-F 0 "#PWR0125" H 1500 6000 50  0001 C CNN
+AR Path="/61005BD4/60A5BF82/60A68DC3" Ref="#PWR0127"  Part="1"
+F 0 "#PWR0127" H 1500 6000 50  0001 C CNN
 F 1 "GND" V 1505 6122 50  0000 R CNN
 F 2 "" H 1500 6250 50  0001 C CNN
@@
 AR Path="/60A48B70/60A6D04A" Ref="#PWR?"  Part="1"
 AR Path="/60A5BF82/60A6D04A" Ref="#PWR?"  Part="1"
-AR Path="/61005BD4/60A5BF82/60A6D04A" Ref="#PWR0136"  Part="1"
-F 0 "#PWR0136" H 4150 6200 50  0001 C CNN
+AR Path="/61005BD4/60A5BF82/60A6D04A" Ref="#PWR0138"  Part="1"
+F 0 "#PWR0138" H 4150 6200 50  0001 C CNN
 F 1 "GND" V 4155 6322 50  0000 R CNN
 F 2 "" H 4150 6450 50  0001 C CNN
@@
 	1    4150 6450
 	0    -1   -1   0
-$EndComp
-$Comp
-L power:+3.3V #PWR?
-U 1 1 60A6DE0B
-P 3600 7350
-AR Path="/60A48B70/60A6DE0B" Ref="#PWR?"  Part="1"
-AR Path="/60A5BF82/60A6DE0B" Ref="#PWR?"  Part="1"
-AR Path="/61005BD4/60A5BF82/60A6DE0B" Ref="#PWR0135"  Part="1"
-F 0 "#PWR0135" H 3600 7200 50  0001 C CNN
-F 1 "+3.3V" H 3615 7523 50  0000 C CNN
-F 2 "" H 3600 7350 50  0001 C CNN
-F 3 "" H 3600 7350 50  0001 C CNN
-	1    3600 7350
-	-1   0    0    1
 $EndComp
 $Comp
@@
 AR Path="/60A48B70/60BC221F" Ref="#PWR?"  Part="1"
 AR Path="/60A5BF82/60BC221F" Ref="#PWR?"  Part="1"
-AR Path="/61005BD4/60A5BF82/60BC221F" Ref="#PWR0120"  Part="1"
-F 0 "#PWR0120" H 1000 850 50  0001 C CNN
+AR Path="/61005BD4/60A5BF82/60BC221F" Ref="#PWR0122"  Part="1"
+F 0 "#PWR0122" H 1000 850 50  0001 C CNN
 F 1 "+3.3VA" H 1015 1173 50  0000 C CNN
 F 2 "" H 1000 1000 50  0001 C CNN
@@
 AR Path="/60A48B70/60BC222B" Ref="#PWR?"  Part="1"
 AR Path="/60A5BF82/60BC222B" Ref="#PWR?"  Part="1"
-AR Path="/61005BD4/60A5BF82/60BC222B" Ref="#PWR0121"  Part="1"
-F 0 "#PWR0121" H 1000 1250 50  0001 C CNN
+AR Path="/61005BD4/60A5BF82/60BC222B" Ref="#PWR0123"  Part="1"
+F 0 "#PWR0123" H 1000 1250 50  0001 C CNN
 F 1 "GND" H 1005 1327 50  0000 C CNN
 F 2 "" H 1000 1500 50  0001 C CNN
@@
 Text GLabel 4950 1000 0    50   Input ~ 0
 ref_dac8
-Text GLabel 3500 1200 0    50   Input ~ 0
-v_out_dac8_a
 $Comp
 L Device:R R?
@@
 ref_dac8
 Text GLabel 3500 2600 0    50   Input ~ 0
-v_out_dac8_b
+v_out_dac8_h
 $Comp
 L Device:R R?
@@
 ref_dac8
 Text GLabel 3500 4000 0    50   Input ~ 0
-v_out_dac8_c
+v_out_dac8_f
 $Comp
 L Amplifier_Operational:TL074 U?
@@
 AR Path="/60A48B70/60BC22F9" Ref="#PWR?"  Part="1"
 AR Path="/60A5BF82/60BC22F9" Ref="#PWR?"  Part="1"
-AR Path="/61005BD4/60A5BF82/60BC22F9" Ref="#PWR0119"  Part="1"
-F 0 "#PWR0119" H 850 5150 50  0001 C CNN
+AR Path="/61005BD4/60A5BF82/60BC22F9" Ref="#PWR0121"  Part="1"
+F 0 "#PWR0121" H 850 5150 50  0001 C CNN
 F 1 "GND" H 855 5227 50  0000 C CNN
 F 2 "" H 850 5400 50  0001 C CNN
@@
 AR Path="/60A48B70/60BC230C" Ref="#PWR?"  Part="1"
 AR Path="/60A5BF82/60BC230C" Ref="#PWR?"  Part="1"
-AR Path="/61005BD4/60A5BF82/60BC230C" Ref="#PWR0118"  Part="1"
-F 0 "#PWR0118" H 850 2800 50  0001 C CNN
+AR Path="/61005BD4/60A5BF82/60BC230C" Ref="#PWR0120"  Part="1"
+F 0 "#PWR0120" H 850 2800 50  0001 C CNN
 F 1 "GND" H 855 2877 50  0000 C CNN
 F 2 "" H 850 3050 50  0001 C CNN
@@
 AR Path="/60A48B70/60BC2320" Ref="#PWR?"  Part="1"
 AR Path="/60A5BF82/60BC2320" Ref="#PWR?"  Part="1"
-AR Path="/61005BD4/60A5BF82/60BC2320" Ref="#PWR0124"  Part="1"
-F 0 "#PWR0124" H 1350 2800 50  0001 C CNN
+AR Path="/61005BD4/60A5BF82/60BC2320" Ref="#PWR0126"  Part="1"
+F 0 "#PWR0126" H 1350 2800 50  0001 C CNN
 F 1 "GND" H 1355 2877 50  0000 C CNN
 F 2 "" H 1350 3050 50  0001 C CNN
@@
 ref_dac8
 Text GLabel 7750 1100 0    50   Input ~ 0
-v_out_dac8_e
+v_out_dac8_a
 $Comp
 L Device:R R?
@@
 ref_dac8
 Text GLabel 7750 2500 0    50   Input ~ 0
-v_out_dac8_f
+v_out_dac8_g
 $Comp
 L Device:R R?
@@
 ref_dac8
 Text GLabel 7750 3900 0    50   Input ~ 0
-v_out_dac8_g
+v_out_dac8_e
 Text Notes 10550 900  0    50   ~ 0
 -5.2V to 5.2V
@@
 ref_dac8
 Text GLabel 7750 5350 0    50   Input ~ 0
-v_out_dac8_h
+v_out_dac8_c
 Text Notes 10550 5150 0    50   ~ 0
 -5.2V to 5.2V
@@
 AR Path="/60A48B70/60CA598A" Ref="#PWR?"  Part="1"
 AR Path="/60A5BF82/60CA598A" Ref="#PWR?"  Part="1"
-AR Path="/61005BD4/60A5BF82/60CA598A" Ref="#PWR0127"  Part="1"
-F 0 "#PWR0127" H 1850 2800 50  0001 C CNN
+AR Path="/61005BD4/60A5BF82/60CA598A" Ref="#PWR0129"  Part="1"
+F 0 "#PWR0129" H 1850 2800 50  0001 C CNN
 F 1 "GND" H 1855 2877 50  0000 C CNN
 F 2 "" H 1850 3050 50  0001 C CNN
@@
 AR Path="/60A48B70/60CA599E" Ref="#PWR?"  Part="1"
 AR Path="/60A5BF82/60CA599E" Ref="#PWR?"  Part="1"
-AR Path="/61005BD4/60A5BF82/60CA599E" Ref="#PWR0132"  Part="1"
-F 0 "#PWR0132" H 2350 2800 50  0001 C CNN
+AR Path="/61005BD4/60A5BF82/60CA599E" Ref="#PWR0134"  Part="1"
+F 0 "#PWR0134" H 2350 2800 50  0001 C CNN
 F 1 "GND" H 2355 2877 50  0000 C CNN
 F 2 "" H 2350 3050 50  0001 C CNN
@@
 Text GLabel 3500 6850 2    50   Input ~ 0
 v_out_dac8_h
-Text HLabel 6350 1100 2    50   Output ~ 0
-dac8_out_a
 Text HLabel 6350 2500 2    50   Output ~ 0
-dac8_out_b
+dac8_out_h
 Text HLabel 6350 3900 2    50   Output ~ 0
-dac8_out_c
+dac8_out_f
 Text HLabel 6350 5350 2    50   Output ~ 0
 dac8_out_d
 Text HLabel 10600 1000 2    50   Output ~ 0
+dac8_out_a
+Text HLabel 10600 2400 2    50   Output ~ 0
+dac8_out_g
+Text HLabel 10600 3800 2    50   Output ~ 0
 dac8_out_e
-Text HLabel 10600 2400 2    50   Output ~ 0
-dac8_out_f
-Text HLabel 10600 3800 2    50   Output ~ 0
-dac8_out_g
 Text HLabel 10600 5250 2    50   Output ~ 0
-dac8_out_h
+dac8_out_c
 Text HLabel 1950 900  0    50   Input ~ 0
 v_ref
@@
 AR Path="/61005BD4/6122FB7F" Ref="#PWR?"  Part="1"
 AR Path="/61005BD4/61028BE5/6122FB7F" Ref="#PWR?"  Part="1"
-AR Path="/61005BD4/60A5BF82/6122FB7F" Ref="#PWR0130"  Part="1"
-F 0 "#PWR0130" H 1950 1250 50  0001 C CNN
+AR Path="/61005BD4/60A5BF82/6122FB7F" Ref="#PWR0132"  Part="1"
+F 0 "#PWR0132" H 1950 1250 50  0001 C CNN
 F 1 "GND" H 1955 1327 50  0000 C CNN
 F 2 "" H 1950 1500 50  0001 C CNN
@@
 	1850 2650 1850 2550
 $Comp
-L power:VCC #PWR0117
+L power:VCC #PWR0119
 U 1 1 611BDDED
 P 850 2550
-F 0 "#PWR0117" H 850 2400 50  0001 C CNN
+F 0 "#PWR0119" H 850 2400 50  0001 C CNN
 F 1 "VCC" H 865 2723 50  0000 C CNN
 F 2 "" H 850 2550 50  0001 C CNN
@@
 $EndComp
 $Comp
-L power:VCC #PWR0123
+L power:VCC #PWR0128
 U 1 1 611BFD6F
 P 1850 2550
-F 0 "#PWR0123" H 1850 2400 50  0001 C CNN
+F 0 "#PWR0128" H 1850 2400 50  0001 C CNN
 F 1 "VCC" H 1865 2723 50  0000 C CNN
 F 2 "" H 1850 2550 50  0001 C CNN
@@
 $EndComp
 $Comp
-L power:VCC #PWR0126
+L power:VCC #PWR0130
 U 1 1 611C033B
 P 1900 4550
-F 0 "#PWR0126" H 1900 4400 50  0001 C CNN
+F 0 "#PWR0130" H 1900 4400 50  0001 C CNN
 F 1 "VCC" H 1915 4723 50  0000 C CNN
 F 2 "" H 1900 4550 50  0001 C CNN
@@
 $EndComp
 $Comp
-L power:VCC #PWR0128
+L power:VCC #PWR0135
 U 1 1 611C0A91
 P 2450 4550
-F 0 "#PWR0128" H 2450 4400 50  0001 C CNN
+F 0 "#PWR0135" H 2450 4400 50  0001 C CNN
 F 1 "VCC" H 2465 4723 50  0000 C CNN
 F 2 "" H 2450 4550 50  0001 C CNN
@@
 $EndComp
 $Comp
-L power:VEE #PWR0129
+L power:VEE #PWR0125
 U 1 1 611C27D3
 P 1350 2550
-F 0 "#PWR0129" H 1350 2400 50  0001 C CNN
+F 0 "#PWR0125" H 1350 2400 50  0001 C CNN
 F 1 "VEE" H 1365 2723 50  0000 C CNN
 F 2 "" H 1350 2550 50  0001 C CNN
@@
 $EndComp
 $Comp
-L power:VEE #PWR0131
+L power:VEE #PWR0133
 U 1 1 611C2BAF
 P 2350 2550
-F 0 "#PWR0131" H 2350 2400 50  0001 C CNN
+F 0 "#PWR0133" H 2350 2400 50  0001 C CNN
 F 1 "VEE" H 2365 2723 50  0000 C CNN
 F 2 "" H 2350 2550 50  0001 C CNN
@@
 $EndComp
 $Comp
-L power:VEE #PWR0133
+L power:VEE #PWR0131
 U 1 1 611C3296
 P 1900 5150
-F 0 "#PWR0133" H 1900 5000 50  0001 C CNN
+F 0 "#PWR0131" H 1900 5000 50  0001 C CNN
 F 1 "VEE" H 1915 5323 50  0000 C CNN
 F 2 "" H 1900 5150 50  0001 C CNN
@@
 $EndComp
 $Comp
-L power:VEE #PWR0134
+L power:VEE #PWR0136
 U 1 1 611C3F9B
 P 2450 5150
-F 0 "#PWR0134" H 2450 5000 50  0001 C CNN
+F 0 "#PWR0136" H 2450 5000 50  0001 C CNN
 F 1 "VEE" H 2465 5323 50  0000 C CNN
 F 2 "" H 2450 5150 50  0001 C CNN
@@
 	-1   0    0    1
 $EndComp
+Text GLabel 3500 1200 0    50   Input ~ 0
+v_out_dac8_b
+Text HLabel 6350 1100 2    50   Output ~ 0
+dac8_out_b
+$Comp
+L power:+3.3VA #PWR0137
+U 1 1 618E7CAA
+P 3600 7350
+F 0 "#PWR0137" H 3600 7200 50  0001 C CNN
+F 1 "+3.3VA" V 3615 7477 50  0000 L CNN
+F 2 "" H 3600 7350 50  0001 C CNN
+F 3 "" H 3600 7350 50  0001 C CNN
+	1    3600 7350
+	-1   0    0    1
+$EndComp

Commit message: Fix issues before manufacturing first prototype
The MIDI jack footprint issue (existent in the first hardware made) is also already fixed in here.
Parts:
- C27, C28, C30, C31, C33, C34: LCSC (none) -> C14663; LCSC Part # (none) -> C14663
- C29: value 3.3u -> 4u7; LCSC (none) -> C19666; LCSC Part # (none) -> C19666
- C32: LCSC (none) -> C15849; LCSC Part # (none) -> C15849
- C35, C36, C37, C38, C39, C40, C41, C42: LCSC (none) -> C1634; LCSC Part # (none) -> C1634
- IC4: LCSC (none) -> C206048; LCSC Part # (none) -> C206048
- R23: LCSC (none) -> C4216; LCSC Part # (none) -> C4216
- R24: LCSC (none) -> C31850; LCSC Part # (none) -> C31850
- R25: LCSC (none) -> C25804; LCSC Part # (none) -> C25804
- R26, R27, R28, R29, R38, R39, R40, R41: LCSC (none) -> C23147; LCSC Part # (none) -> C23147
- R30, R31, R32, R33, R42, R43, R44, R45: LCSC (none) -> C22807; LCSC Part # (none) -> C22807
- R34, R35, R36, R37, R46, R47, R48, R49: LCSC (none) -> C21190; LCSC Part # (none) -> C21190
- U5, U6: LCSC (none) -> C96507; LCSC Part # (none) -> C96507

Commit message: wire up ad5328
Parts:
- removed IC4: DAC5578SPWR, SOP65P640X120-16N, symbol DAC5578SPWR:DAC5578SPWR
- removed R25: 10k, Resistor_SMD:R_0603_1608Metric, symbol Device:R
- added IC4: AD5328BRUZ, SOP65P640X120-16N, symbol AD5328BRUZ:AD5328BRUZ
- C29: value 4u7 -> 10u; LCSC C19666 -> C19702; LCSC Part # C19666 -> C19702
Connections:
- net labels added: dac8_css
- wire segments 154 -> 149
Changed lines of the file:
@@
 $EndDescr
-$Comp
-L DAC5578SPWR:DAC5578SPWR IC4
-U 1 1 60A5C8AD
-P 1800 6250
-F 0 "IC4" H 2650 6515 50  0000 C CNN
-F 1 "DAC5578SPWR" H 2650 6424 50  0000 C CNN
-F 2 "SOP65P640X120-16N" H 3350 6350 50  0001 L CNN
-F 3 "http://www.ti.com/lit/gpn/DAC5578" H 3350 6250 50  0001 L CNN
-F 4 "8-bit, Octal Channel, Ultra-Low Glitch, Voltage Output, 2-Wire Interface DAC" H 3350 6150 50  0001 L CNN "Description"
-F 5 "" H 3350 6050 50  0001 L CNN "Height"
-F 6 "Texas Instruments" H 3350 5950 50  0001 L CNN "Manufacturer_Name"
-F 7 "DAC5578SPWR" H 3350 5850 50  0001 L CNN "Manufacturer_Part_Number"
-F 8 "595-DAC5578SPWR" H 3350 5750 50  0001 L CNN "Mouser Part Number"
-F 9 "https://www.mouser.co.uk/ProductDetail/Texas-Instruments/DAC5578SPWR?qs=EuM%2FBx4ov4S16BMU6rn1hg%3D%3D" H 3350 5650 50  0001 L CNN "Mouser Price/Stock"
-F 10 "DAC5578SPWR" H 3350 5550 50  0001 L CNN "Arrow Part Number"
-F 11 "https://www.arrow.com/en/products/dac5578spwr/texas-instruments" H 3350 5450 50  0001 L CNN "Arrow Price/Stock"
-F 12 "C206048" H 1800 6250 50  0001 C CNN "LCSC Part #"
-F 13 "C206048" H 1800 6250 50  0001 C CNN "LCSC"
-	1    1800 6250
-	1    0    0    -1
-$EndComp
 $Comp
 L power:+3.3VA #PWR0124
 U 1 1 60A68DBC
-P 1300 6450
-F 0 "#PWR0124" H 1300 6300 50  0001 C CNN
-F 1 "+3.3VA" V 1315 6577 50  0000 L CNN
-F 2 "" H 1300 6450 50  0001 C CNN
-F 3 "" H 1300 6450 50  0001 C CNN
-	1    1300 6450
+P 1400 6400
+F 0 "#PWR0124" H 1400 6250 50  0001 C CNN
+F 1 "+3.3VA" V 1415 6527 50  0000 L CNN
+F 2 "" H 1400 6400 50  0001 C CNN
+F 3 "" H 1400 6400 50  0001 C CNN
+	1    1400 6400
 	0    -1   -1   0
 $EndComp
 Wire Wire Line
-	1300 6450 1800 6450
-Wire Wire Line
-	1800 6350 1650 6350
-Wire Wire Line
-	1650 6250 1800 6250
-Wire Wire Line
-	1500 6250 1650 6250
-Connection ~ 1650 6250
-Wire Wire Line
-	1650 6350 1650 6250
+	1400 6400 1900 6400
 $Comp
 L power:GND #PWR?
 U 1 1 60A68DC3
-P 1500 6250
+P 1550 6200
 AR Path="/60A48B70/60A68DC3" Ref="#PWR?"  Part="1"
 AR Path="/60A5BF82/60A68DC3" Ref="#PWR?"  Part="1"
 AR Path="/61005BD4/60A5BF82/60A68DC3" Ref="#PWR0127"  Part="1"
-F 0 "#PWR0127" H 1500 6000 50  0001 C CNN
-F 1 "GND" V 1505 6122 50  0000 R CNN
-F 2 "" H 1500 6250 50  0001 C CNN
-F 3 "" H 1500 6250 50  0001 C CNN
-	1    1500 6250
+F 0 "#PWR0127" H 1550 5950 50  0001 C CNN
+F 1 "GND" V 1555 6072 50  0000 R CNN
+F 2 "" H 1550 6200 50  0001 C CNN
+F 3 "" H 1550 6200 50  0001 C CNN
+	1    1550 6200
 	0    1    1    0
 $EndComp
@@
 L power:GND #PWR?
 U 1 1 60A6D04A
-P 4150 6450
+P 4050 6400
 AR Path="/60A48B70/60A6D04A" Ref="#PWR?"  Part="1"
 AR Path="/60A5BF82/60A6D04A" Ref="#PWR?"  Part="1"
 AR Path="/61005BD4/60A5BF82/60A6D04A" Ref="#PWR0138"  Part="1"
-F 0 "#PWR0138" H 4150 6200 50  0001 C CNN
-F 1 "GND" V 4155 6322 50  0000 R CNN
-F 2 "" H 4150 6450 50  0001 C CNN
-F 3 "" H 4150 6450 50  0001 C CNN
-	1    4150 6450
+F 0 "#PWR0138" H 4050 6150 50  0001 C CNN
+F 1 "GND" V 4055 6272 50  0000 R CNN
+F 2 "" H 4050 6400 50  0001 C CNN
+F 3 "" H 4050 6400 50  0001 C CNN
+	1    4050 6400
 	0    -1   -1   0
 $EndComp
-$Comp
-L Device:R R25
-U 1 1 60A6F434
-P 3600 7200
-F 0 "R25" H 3530 7154 50  0000 R CNN
-F 1 "10k" H 3530 7245 50  0000 R CNN
-F 2 "Resistor_SMD:R_0603_1608Metric" V 3530 7200 50  0001 C CNN
-F 3 "~" H 3600 7200 50  0001 C CNN
-F 4 "C25804" H 3600 7200 50  0001 C CNN "LCSC Part #"
-F 5 "C25804" H 3600 7200 50  0001 C CNN "LCSC"
-	1    3600 7200
-	-1   0    0    1
-$EndComp
-Wire Wire Line
-	3500 6950 3600 6950
-Wire Wire Line
-	3600 6950 3600 7050
-Text HLabel 3500 6250 2    50   Input ~ 0
+Text HLabel 3400 6200 2    50   Input ~ 0
 dac8_scl
-Text HLabel 3500 6350 2    50   BiDi ~ 0
-dac8_sda
-Wire Wire Line
-	3500 6450 4150 6450
+Wire Wire Line
+	3400 6400 4050 6400
 $Comp
 L power:+3.3VA #PWR?
@@
 AR Path="/61005BD4/60A5BF82/60BC2231" Ref="C29"  Part="1"
 F 0 "C29" H 1315 1296 50  0000 L CNN
-F 1 "4u7" H 1315 1205 50  0000 L CNN
+F 1 "10u" H 1315 1205 50  0000 L CNN
 F 2 "Capacitor_SMD:C_0603_1608Metric" H 1238 1100 50  0001 C CNN
 F 3 "~" H 1200 1250 50  0001 C CNN
-F 4 "C19666" H 1200 1250 50  0001 C CNN "LCSC Part #"
-F 5 "C19666" H 1200 1250 50  0001 C CNN "LCSC"
+F 4 "C19702" H 1200 1250 50  0001 C CNN "LCSC Part #"
+F 5 "C19702" H 1200 1250 50  0001 C CNN "LCSC"
 	1    1200 1250
 	1    0    0    -1
@@
 Text GLabel 4950 2400 0    50   Input ~ 0
 ref_dac8
-Text GLabel 3500 2600 0    50   Input ~ 0
-v_out_dac8_h
 $Comp
 L Device:R R?
@@
 Text GLabel 4950 3800 0    50   Input ~ 0
 ref_dac8
-Text GLabel 3500 4000 0    50   Input ~ 0
-v_out_dac8_f
 $Comp
 L Amplifier_Operational:TL074 U?
@@
 ref_dac8
 Text GLabel 3500 5450 0    50   Input ~ 0
-v_out_dac8_d
+v_out_dac8_c
 Text Notes 6300 5250 0    50   ~ 0
 -5.2V to 5.2V
@@
 ref_dac8
 Text GLabel 7750 1100 0    50   Input ~ 0
-v_out_dac8_a
+v_out_dac8_e
 $Comp
 L Device:R R?
@@
 ref_dac8
 Text GLabel 7750 2500 0    50   Input ~ 0
-v_out_dac8_g
+v_out_dac8_h
 $Comp
 L Device:R R?
@@
 ref_dac8
 Text GLabel 7750 3900 0    50   Input ~ 0
-v_out_dac8_e
+v_out_dac8_g
 Text Notes 10550 900  0    50   ~ 0
 -5.2V to 5.2V
@@
 ref_dac8
 Text GLabel 7750 5350 0    50   Input ~ 0
-v_out_dac8_c
+v_out_dac8_f
 Text Notes 10550 5150 0    50   ~ 0
 -5.2V to 5.2V
@@
 Wire Wire Line
 	9850 2400 9800 2400
-Text GLabel 1800 6550 0    50   Input ~ 0
+Text GLabel 1900 6500 0    50   Input ~ 0
 v_out_dac8_a
-Text GLabel 1800 6650 0    50   Input ~ 0
+Text GLabel 1900 6700 0    50   Input ~ 0
 v_out_dac8_c
-Text GLabel 1800 6750 0    50   Input ~ 0
+Text GLabel 3400 6800 2    50   Input ~ 0
 v_out_dac8_e
-Text GLabel 1800 6850 0    50   Input ~ 0
+Text GLabel 3400 6600 2    50   Input ~ 0
 v_out_dac8_g
-Text GLabel 3500 6550 2    50   Input ~ 0
+Text GLabel 1900 6600 0    50   Input ~ 0
 v_out_dac8_b
-Text GLabel 3500 6650 2    50   Input ~ 0
+Text GLabel 1900 6800 0    50   Input ~ 0
 v_out_dac8_d
-Text GLabel 3500 6750 2    50   Input ~ 0
+Text GLabel 3400 6700 2    50   Input ~ 0
 v_out_dac8_f
-Text GLabel 3500 6850 2    50   Input ~ 0
+Text GLabel 3400 6500 2    50   Input ~ 0
 v_out_dac8_h
-Text HLabel 6350 2500 2    50   Output ~ 0
+Text HLabel 6350 5350 2    50   Output ~ 0
+dac8_out_c
+Text HLabel 10600 1000 2    50   Output ~ 0
+dac8_out_e
+Text HLabel 10600 2400 2    50   Output ~ 0
 dac8_out_h
-Text HLabel 6350 3900 2    50   Output ~ 0
+Text HLabel 10600 5250 2    50   Output ~ 0
 dac8_out_f
-Text HLabel 6350 5350 2    50   Output ~ 0
-dac8_out_d
-Text HLabel 10600 1000 2    50   Output ~ 0
-dac8_out_a
-Text HLabel 10600 2400 2    50   Output ~ 0
-dac8_out_g
-Text HLabel 10600 3800 2    50   Output ~ 0
-dac8_out_e
-Text HLabel 10600 5250 2    50   Output ~ 0
-dac8_out_c
 Text HLabel 1950 900  0    50   Input ~ 0
 v_ref
@@
 	2350 900  2350 1050
 Connection ~ 2350 1050
-Text GLabel 1800 6950 0    50   Input ~ 0
+Text GLabel 1900 6900 0    50   Input ~ 0
 v_ref_dac8
 Wire Wire Line
@@
 	-1   0    0    1
 $EndComp
-Text GLabel 3500 1200 0    50   Input ~ 0
+Text GLabel 3400 6900 2    50   Input ~ 0
+v_ref_dac8
+Text HLabel 6350 3900 2    50   Output ~ 0
+dac8_out_b
+Text GLabel 3500 4000 0    50   Input ~ 0
 v_out_dac8_b
 Text HLabel 6350 1100 2    50   Output ~ 0
-dac8_out_b
-$Comp
-L power:+3.3VA #PWR0137
-U 1 1 618E7CAA
-P 3600 7350
-F 0 "#PWR0137" H 3600 7200 50  0001 C CNN
-F 1 "+3.3VA" V 3615 7477 50  0000 L CNN
-F 2 "" H 3600 7350 50  0001 C CNN
-F 3 "" H 3600 7350 50  0001 C CNN
-	1    3600 7350
-	-1   0    0    1
-$EndComp
+dac8_out_d
+Text GLabel 3500 1200 0    50   Input ~ 0
+v_out_dac8_d
+Text HLabel 6350 2500 2    50   Output ~ 0
+dac8_out_a
+Wire Wire Line
+	1550 6200 1900 6200
+Text HLabel 3400 6300 2    50   Input ~ 0
+dac8_sda
+Text HLabel 1900 6300 0    50   Input ~ 0
+dac8_css
+$Comp
+L AD5328BRUZ:AD5328BRUZ IC4
+U 1 1 61AB2D74
+P 1900 6200
+F 0 "IC4" H 2650 6465 50  0000 C CNN
+F 1 "AD5328BRUZ" H 2650 6374 50  0000 C CNN
+F 2 "SOP65P640X120-16N" H 3250 6300 50  0001 L CNN
+F 3 "http://www.analog.com/static/imported-files/data_sheets/AD5308_5318_5328.pdf" H 3250 6200 50  0001 L CNN
+F 4 "AD5328BRUZ, 12-Bit General Purpose DAC 8-channel 167ksps, SPI, Microwire, 16-Pin TSSOP" H 3250 6100 50  0001 L CNN "Description"
+F 5 "1.2" H 3250 6000 50  0001 L CNN "Height"
+F 6 "Analog Devices" H 3250 5900 50  0001 L CNN "Manufacturer_Name"
+F 7 "AD5328BRUZ" H 3250 5800 50  0001 L CNN "Manufacturer_Part_Number"
+F 8 "584-AD5328BRUZ" H 3250 5700 50  0001 L CNN "Mouser Part Number"
+F 9 "https://www.mouser.com/Search/Refine.aspx?Keyword=584-AD5328BRUZ" H 3250 5600 50  0001 L CNN "Mouser Price/Stock"
+F 10 "AD5328BRUZ" H 3250 5500 50  0001 L CNN "Arrow Part Number"
+F 11 "https://www.arrow.com/en/products/ad5328bruz/analog-devices" H 3250 5400 50  0001 L CNN "Arrow Price/Stock"
+F 12 "C29162" H 1900 6200 50  0001 C CNN "LCSC"
+	1    1900 6200
+	1    0    0    -1
+$EndComp
+Text GLabel 3500 2600 0    50   Input ~ 0
+v_out_dac8_a
+Text HLabel 10600 3800 2    50   Output ~ 0
+dac8_out_g
 $EndSCHEMATC
