File: hardware/midi2cv-front.sch (KiCad schematic (older format))
At the start: 26 parts

Commit message: Move to single schema tree
Parts:
- added IC?: LP5012PWR, SOP65P640X120-24N, symbol LP5012PWR:LP5012PWR
Changed lines of the file:
@@
 $Descr A4 11693 8268
 encoding utf-8
-Sheet 1 1
+Sheet 5 5
 Title ""
 Date ""
@@
 AR Path="/60A44BB1/60A45791" Ref="U?"  Part="1"
 AR Path="/60A45791" Ref="U?"  Part="1"
+AR Path="/61006ED6/60A45791" Ref="U?"  Part="1"
 F 0 "U?" H 3450 2217 50  0000 C CNN
 F 1 "6N137" H 3450 2126 50  0000 C CNN
@@
 Wire Wire Line
 	3850 1550 4000 1550
+$Comp
+L LP5012PWR:LP5012PWR IC?
+U 1 1 6100A408
+P 2900 4050
+F 0 "IC?" H 3500 4315 50  0000 C CNN
+F 1 "LP5012PWR" H 3500 4224 50  0000 C CNN
+F 2 "SOP65P640X120-24N" H 3950 4150 50  0001 L CNN
+F 3 "https://www.ti.com/lit/ds/symlink/lp5012.pdf?ts=1615929314042&ref_url=https%253A%252F%252Fwww.mouser.co.uk%252F" H 3950 4050 50  0001 L CNN
+F 4 "LED Lighting Drivers" H 3950 3950 50  0001 L CNN "Description"
+F 5 "1.2" H 3950 3850 50  0001 L CNN "Height"
+F 6 "Texas Instruments" H 3950 3750 50  0001 L CNN "Manufacturer_Name"
+F 7 "LP5012PWR" H 3950 3650 50  0001 L CNN "Manufacturer_Part_Number"
+F 8 "595-LP5012PWR" H 3950 3550 50  0001 L CNN "Mouser Part Number"
+F 9 "https://www.mouser.co.uk/ProductDetail/Texas-Instruments/LP5012PWR?qs=T94vaHKWudSL6jLwBy12Hg%3D%3D" H 3950 3450 50  0001 L CNN "Mouser Price/Stock"
+F 10 "" H 3950 3350 50  0001 L CNN "Arrow Part Number"
+F 11 "" H 3950 3250 50  0001 L CNN "Arrow Price/Stock"
+	1    2900 4050
+	1    0    0    -1
+$EndComp
 $EndSCHEMATC

Commit message: First preliminary board design
Parts:
- removed C?: 100n, symbol Device:C
- removed D?: 1N4148, Diode_THT:D_DO-35_SOD27_P7.62mm_Horizontal, symbol Diode:1N4148
- removed IC?: LP5012PWR, SOP65P640X120-24N, symbol LP5012PWR:LP5012PWR
- removed J? (x20): PJ398SM-12, THONK_PJ398SM-12, symbol PJ398SM-12:PJ398SM-12
- removed J?: SD-50BV, SD-50BV, symbol SD-50BV:SD-50BV
- removed R?: 220R, symbol Device:R
- removed R?: 10k, symbol Device:R
- removed U?: 6N137, Package_DIP:DIP-8_W7.62mm, symbol Isolator:6N137
- added D1: BAT54S, Package_TO_SOT_SMD:SOT-23, symbol Diode:BAT54S
- added J10, J11, J12, J13, J14, J15, J16, J17, J18, J19, J20, J21, J22, J23, J24, J25, J26, J27, J28, J29, J8, J9: PJ398SM, Connector_Audio:Jack_3.5mm_QingPu_WQP-PJ398SM_Vertical_CircularHoles, symbol Connector:AudioJack2_SwitchT
- added J7: SD-50BV, SD-50BV:SD-50BV, symbol SD-50BV:SD-50BV
- added R1, R2: 100k, Resistor_SMD:R_0603_1608Metric, symbol Device:R
- added S1, S2, S3, S4: TC002-N11AS1XKT-RGB, TC002-N11AS1XKT-RGB:TC002N11AS1XKTRGB, symbol TC002-N11AS1XKT-RGB:TC002-N11AS1XKT-RGB
Connections:
- net labels added: 1_16_out, button_a, button_b, button_c, button_d, clock_out, cv_in_a, cv_in_b, dac4_out_a, dac4_out_b, dac4_out_c, dac4_out_d, dac8_out_a, dac8_out_b, dac8_out_c, dac8_out_d, dac8_out_e, dac8_out_f, dac8_out_g, dac8_out_h, gate_out_a, gate_out_b, gate_out_c, gate_out_d, jack_detect, led_out_a_b, led_out_a_g, led_out_a_r, led_out_b_b, led_out_b_g, led_out_b_r, led_out_c_b, led_out_c_g, led_out_c_r, led_out_d_b, led_out_d_g, led_out_d_r, midi_in+, midi_in-, run_out, var_out
- net labels removed: midi_rx
- wire segments 16 -> 32
- no-connect marks 4 -> 3
Other:
- note added: "1&2 are connected to 3&4 when button is pressed"

Commit message: Layed out stretched design
Parts:
- renumbered J8 to J10, J9 to J11, J10 to J12, J11 to J13, J12 to J14, J13 to J15, J14 to J16, J15 to J17, J16 to J18, J17 to J19, J18 to J20, J19 to J21, J20 to J22, J21 to J23, J22 to J24, J23 to J25, J24 to J26, J25 to J27, J26 to J28, J27 to J29, J28 to J30, J29 to J31, J7 to J9

Commit message: Fix issues before manufacturing first prototype
The MIDI jack footprint issue (existent in the first hardware made) is also already fixed in here.
Parts:
- D1: LCSC (none) -> C571351; LCSC Part # (none) -> C571351
Connections:
- net midi_in+: now also J9.2; no longer J9.4
- net midi_in-: now also J9.4; no longer J9.5
Changed lines of the file:
@@
 F 2 "Package_TO_SOT_SMD:SOT-23" H 9375 5925 50  0001 L CNN
 F 3 "https://www.diodes.com/assets/Datasheets/ds11005.pdf" H 9180 5800 50  0001 C CNN
+F 4 "C571351" H 9300 5800 50  0001 C CNN "LCSC Part #"
+F 5 "C571351" H 9300 5800 50  0001 C CNN "LCSC"
 	1    9300 5800
 	1    0    0    -1
@@
 $EndComp
 NoConn ~ 2500 6350
-NoConn ~ 2500 6450
+NoConn ~ 3300 6450
 NoConn ~ 2500 6550
+Text HLabel 2500 6450 0    50   Output ~ 0
+midi_in+
 Text HLabel 3300 6350 2    50   Output ~ 0
-midi_in+
-Text HLabel 3300 6450 2    50   Output ~ 0
 midi_in-
 $EndSCHEMATC

Commit message: Fix jack switches connected to ground
Connections:
- net GND: no longer J10.TN, J11.TN, J12.TN, J13.TN, J14.TN, J16.TN, J17.TN, J18.TN, J19.TN, J20.TN, J22.TN, J23.TN, J24.TN, J25.TN, J26.TN, J27.TN, J28.TN, J29.TN, J30.TN, J31.TN
- no-connect marks 3 -> 24
