File: hardware/power_ref.sch (KiCad schematic (older format))
At the start: 23 parts, among them IC5 ADP150AUJZ-3.3-R7, J31 Eurorack PWR, U7 LM1117-3.3, U8 LM1117-5.0, U9 LM4040DBZ-10

Commit message: Layed out stretched design
Parts:
- renumbered J31 to J33
Changed lines of the file:
@@
 	8350 1550 8350 1750
 $Comp
-L power:GND #PWR0159
+L power:GND #PWR0161
 U 1 1 5FDFEFF3
 P 8350 2400
-F 0 "#PWR0159" H 8350 2150 50  0001 C CNN
+F 0 "#PWR0161" H 8350 2150 50  0001 C CNN
 F 1 "GND" H 8355 2227 50  0000 C CNN
 F 2 "" H 8350 2400 50  0001 C CNN
@@
 Connection ~ 8350 1550
 $Comp
-L power:GND #PWR0160
+L power:GND #PWR0162
 U 1 1 5FDFF00B
 P 9200 2400
-F 0 "#PWR0160" H 9200 2150 50  0001 C CNN
+F 0 "#PWR0162" H 9200 2150 50  0001 C CNN
 F 1 "GND" H 9205 2227 50  0000 C CNN
 F 2 "" H 9200 2400 50  0001 C CNN
@@
 -10V reference
 $Comp
-L power:VEE #PWR0156
+L power:VEE #PWR0158
 U 1 1 5FDFF018
 P 7500 1350
-F 0 "#PWR0156" H 7500 1200 50  0001 C CNN
+F 0 "#PWR0158" H 7500 1200 50  0001 C CNN
 F 1 "VEE" H 7515 1523 50  0000 C CNN
 F 2 "" H 7500 1350 50  0001 C CNN
@@
 0.1mA
 $Comp
-L power:VCC #PWR0138
+L power:VCC #PWR0140
 U 1 1 5FDFF026
 P 1600 4050
-F 0 "#PWR0138" H 1600 3900 50  0001 C CNN
+F 0 "#PWR0140" H 1600 3900 50  0001 C CNN
 F 1 "VCC" V 1618 4177 50  0000 L CNN
 F 2 "" H 1600 4050 50  0001 C CNN
@@
 	2450 4050 2650 4050
 $Comp
-L power:+5V #PWR0152
+L power:+5V #PWR0154
 U 1 1 5FDFF049
 P 4500 4050
-F 0 "#PWR0152" H 4500 3900 50  0001 C CNN
+F 0 "#PWR0154" H 4500 3900 50  0001 C CNN
 F 1 "+5V" H 4515 4223 50  0000 C CNN
 F 2 "" H 4500 4050 50  0001 C CNN
@@
 $EndComp
 $Comp
-L power:GND #PWR0149
+L power:GND #PWR0151
 U 1 1 5FDFF04F
 P 3950 4350
-F 0 "#PWR0149" H 3950 4100 50  0001 C CNN
+F 0 "#PWR0151" H 3950 4100 50  0001 C CNN
 F 1 "GND" H 3955 4177 50  0000 C CNN
 F 2 "" H 3950 4350 50  0001 C CNN
@@
 $EndComp
 $Comp
-L power:GND #PWR0153
+L power:GND #PWR0155
 U 1 1 5FDFF05E
 P 4500 4350
-F 0 "#PWR0153" H 4500 4100 50  0001 C CNN
+F 0 "#PWR0155" H 4500 4100 50  0001 C CNN
 F 1 "GND" H 4505 4177 50  0000 C CNN
 F 2 "" H 4500 4350 50  0001 C CNN
@@
 $EndComp
 $Comp
-L power:GND #PWR0144
+L power:GND #PWR0146
 U 1 1 5FDFF064
 P 2650 4350
-F 0 "#PWR0144" H 2650 4100 50  0001 C CNN
+F 0 "#PWR0146" H 2650 4100 50  0001 C CNN
 F 1 "GND" H 2655 4177 50  0000 C CNN
 F 2 "" H 2650 4350 50  0001 C CNN
@@
 $EndComp
 $Comp
-L power:GND #PWR0142
+L power:GND #PWR0144
 U 1 1 5FDFF06A
 P 1950 4350
-F 0 "#PWR0142" H 1950 4100 50  0001 C CNN
+F 0 "#PWR0144" H 1950 4100 50  0001 C CNN
 F 1 "GND" H 1955 4177 50  0000 C CNN
 F 2 "" H 1950 4350 50  0001 C CNN
@@
 $EndComp
 $Comp
-L power:GND #PWR0146
+L power:GND #PWR0148
 U 1 1 5FDFF076
 P 3300 4350
-F 0 "#PWR0146" H 3300 4100 50  0001 C CNN
+F 0 "#PWR0148" H 3300 4100 50  0001 C CNN
 F 1 "GND" H 3305 4177 50  0000 C CNN
 F 2 "" H 3300 4350 50  0001 C CNN
@@
 $EndComp
 $Comp
-L Connector_Generic:Conn_02x05_Odd_Even J31
+L Connector_Generic:Conn_02x05_Odd_Even J33
 U 1 1 5FDFF083
 P 2050 1900
-F 0 "J31" H 2100 2317 50  0000 C CNN
+F 0 "J33" H 2100 2317 50  0000 C CNN
 F 1 "Eurorack PWR" H 2100 2226 50  0000 C CNN
 F 2 "Connector_IDC:IDC-Header_2x05_P2.54mm_Vertical" H 2050 1900 50  0001 C CNN
@@
 Connection ~ 1850 2000
 $Comp
-L power:GND #PWR0139
+L power:GND #PWR0141
 U 1 1 5FDFF093
 P 1700 1900
-F 0 "#PWR0139" H 1700 1650 50  0001 C CNN
+F 0 "#PWR0141" H 1700 1650 50  0001 C CNN
 F 1 "GND" V 1705 1772 50  0000 R CNN
 F 2 "" H 1700 1900 50  0001 C CNN
@@
 $EndComp
 $Comp
-L power:-12V #PWR0140
+L power:-12V #PWR0142
 U 1 1 5FDFF0A8
 P 1850 1700
-F 0 "#PWR0140" H 1850 1800 50  0001 C CNN
+F 0 "#PWR0142" H 1850 1800 50  0001 C CNN
 F 1 "-12V" V 1865 1828 50  0000 L CNN
 F 2 "" H 1850 1700 50  0001 C CNN
@@
 Connection ~ 1850 1700
 $Comp
-L power:+12V #PWR0141
+L power:+12V #PWR0143
 U 1 1 5FDFF0AF
 P 1850 2100
-F 0 "#PWR0141" H 1850 1950 50  0001 C CNN
+F 0 "#PWR0143" H 1850 1950 50  0001 C CNN
 F 1 "+12V" V 1865 2228 50  0000 L CNN
 F 2 "" H 1850 2100 50  0001 C CNN
@@
 Connection ~ 2350 2000
 $Comp
-L power:GND #PWR0154
+L power:GND #PWR0156
 U 1 1 5FDFF0BB
 P 4750 1900
-F 0 "#PWR0154" H 4750 1650 50  0001 C CNN
+F 0 "#PWR0156" H 4750 1650 50  0001 C CNN
 F 1 "GND" V 4755 1772 50  0000 R CNN
 F 2 "" H 4750 1900 50  0001 C CNN
@@
 	3750 2100 4050 2100
 $Comp
-L power:VEE #PWR0150
+L power:VEE #PWR0152
 U 1 1 5FDFF0D1
 P 4050 1450
-F 0 "#PWR0150" H 4050 1300 50  0001 C CNN
+F 0 "#PWR0152" H 4050 1300 50  0001 C CNN
 F 1 "VEE" H 4067 1623 50  0000 C CNN
 F 2 "" H 4050 1450 50  0001 C CNN
@@
 	10200 2750 10200 1000
 $Comp
-L power:+5V #PWR0137
+L power:+5V #PWR0139
 U 1 1 5FDFF10A
 P 1400 6150
-F 0 "#PWR0137" H 1400 6000 50  0001 C CNN
+F 0 "#PWR0139" H 1400 6000 50  0001 C CNN
 F 1 "+5V" V 1415 6278 50  0000 L CNN
 F 2 "" H 1400 6150 50  0001 C CNN
@@
 Connection ~ 2750 6150
 $Comp
-L power:GND #PWR0145
+L power:GND #PWR0147
 U 1 1 5FDFF11D
 P 2750 6450
-F 0 "#PWR0145" H 2750 6200 50  0001 C CNN
+F 0 "#PWR0147" H 2750 6200 50  0001 C CNN
 F 1 "GND" H 2755 6277 50  0000 C CNN
 F 2 "" H 2750 6450 50  0001 C CNN
@@
 $EndComp
 $Comp
-L power:GND #PWR0147
+L power:GND #PWR0149
 U 1 1 5FDFF123
 P 3450 6450
-F 0 "#PWR0147" H 3450 6200 50  0001 C CNN
+F 0 "#PWR0149" H 3450 6200 50  0001 C CNN
 F 1 "GND" H 3455 6277 50  0000 C CNN
 F 2 "" H 3450 6450 50  0001 C CNN
@@
 $EndComp
 $Comp
-L power:GND #PWR0143
+L power:GND #PWR0145
 U 1 1 5FDFF12F
 P 2000 6450
-F 0 "#PWR0143" H 2000 6200 50  0001 C CNN
+F 0 "#PWR0145" H 2000 6200 50  0001 C CNN
 F 1 "GND" H 2005 6277 50  0000 C CNN
 F 2 "" H 2000 6450 50  0001 C CNN
@@
 	3450 6150 3800 6150
 $Comp
-L power:+3V3 #PWR0148
+L power:+3V3 #PWR0150
 U 1 1 5FE03B05
 P 3800 6150
-F 0 "#PWR0148" H 3800 6000 50  0001 C CNN
+F 0 "#PWR0150" H 3800 6000 50  0001 C CNN
 F 1 "+3V3" V 3815 6278 50  0000 L CNN
 F 2 "" H 3800 6150 50  0001 C CNN
@@
 +3.3VA Voltage Regulator
 $Comp
-L power:+5V #PWR0155
+L power:+5V #PWR0157
 U 1 1 5FEA3E47
 P 7450 4000
-F 0 "#PWR0155" H 7450 3850 50  0001 C CNN
+F 0 "#PWR0157" H 7450 3850 50  0001 C CNN
 F 1 "+5V" V 7465 4128 50  0000 L CNN
 F 2 "" H 7450 4000 50  0001 C CNN
@@
 $EndComp
 $Comp
-L power:GND #PWR0158
+L power:GND #PWR0160
 U 1 1 5FEB2A32
 P 7750 4350
-F 0 "#PWR0158" H 7750 4100 50  0001 C CNN
+F 0 "#PWR0160" H 7750 4100 50  0001 C CNN
 F 1 "GND" H 7755 4177 50  0000 C CNN
 F 2 "" H 7750 4350 50  0001 C CNN
@@
 AR Path="/5FEBC275" Ref="#PWR?"  Part="1"
 AR Path="/5FDE753F/5FEBC275" Ref="#PWR?"  Part="1"
-AR Path="/61005BD4/6102A76E/5FEBC275" Ref="#PWR0162"  Part="1"
-F 0 "#PWR0162" H 9850 3950 50  0001 C CNN
+AR Path="/61005BD4/6102A76E/5FEBC275" Ref="#PWR0164"  Part="1"
+F 0 "#PWR0164" H 9850 3950 50  0001 C CNN
 F 1 "+3.3VA" V 9865 4228 50  0000 L CNN
 F 2 "" H 9850 4100 50  0001 C CNN
@@
 	9600 4100 9850 4100
 $Comp
-L power:GND #PWR0161
+L power:GND #PWR0163
 U 1 1 5FEBEC47
 P 9600 4400
-F 0 "#PWR0161" H 9600 4150 50  0001 C CNN
+F 0 "#PWR0163" H 9600 4150 50  0001 C CNN
 F 1 "GND" H 9605 4227 50  0000 C CNN
 F 2 "" H 9600 4400 50  0001 C CNN
@@
 Connection ~ 2350 2100
 $Comp
-L power:VCC #PWR0151
+L power:VCC #PWR0153
 U 1 1 5FF4123A
 P 4050 2350
-F 0 "#PWR0151" H 4050 2200 50  0001 C CNN
+F 0 "#PWR0153" H 4050 2200 50  0001 C CNN
 F 1 "VCC" V 4068 2477 50  0000 L CNN
 F 2 "" H 4050 2350 50  0001 C CNN
@@
 Connection ~ 7500 1550
 $Comp
-L power:GND #PWR0157
+L power:GND #PWR0159
 U 1 1 5FE95D6C
 P 7500 2400
-F 0 "#PWR0157" H 7500 2150 50  0001 C CNN
+F 0 "#PWR0159" H 7500 2150 50  0001 C CNN
 F 1 "GND" H 7505 2227 50  0000 C CNN
 F 2 "" H 7500 2400 50  0001 C CNN

Commit message: Fix issues before manufacturing first prototype
The MIDI jack footprint issue (existent in the first hardware made) is also already fixed in here.
Parts:
- IC5: LCSC (none) -> C29149; LCSC Part # (none) -> C29149
- U8: LCSC (none) -> C6187; LCSC Part # (none) -> C6187
- U9: LCSC (none) -> C201738; LCSC Part # (none) -> C201738
Changed lines of the file:
@@
 F 2 "Package_TO_SOT_SMD:SOT-23" H 8350 1700 50  0001 C CIN
 F 3 "http://www.ti.com/lit/ds/symlink/lm4040-n.pdf" H 8350 1900 50  0001 C CIN
+F 4 "C201738" H 8350 1900 50  0001 C CNN "LCSC Part #"
+F 5 "C201738" H 8350 1900 50  0001 C CNN "LCSC"
 	1    8350 1900
 	0    1    1    0
@@
 	1850 2000 1850 1900
 Connection ~ 1850 2000
-$Comp
-L power:GND #PWR0141
-U 1 1 5FDFF093
-P 1700 1900
-F 0 "#PWR0141" H 1700 1650 50  0001 C CNN
-F 1 "GND" V 1705 1772 50  0000 R CNN
-F 2 "" H 1700 1900 50  0001 C CNN
-F 3 "" H 1700 1900 50  0001 C CNN
-	1    1700 1900
-	0    1    1    0
-$EndComp
 Wire Wire Line
 	1850 1900 1700 1900
@@
 L power:-12V #PWR0142
 U 1 1 5FDFF0A8
-P 1850 1700
-F 0 "#PWR0142" H 1850 1800 50  0001 C CNN
-F 1 "-12V" V 1865 1828 50  0000 L CNN
-F 2 "" H 1850 1700 50  0001 C CNN
-F 3 "" H 1850 1700 50  0001 C CNN
-	1    1850 1700
+P 1550 1700
+F 0 "#PWR0142" H 1550 1800 50  0001 C CNN
+F 1 "-12V" V 1565 1828 50  0000 L CNN
+F 2 "" H 1550 1700 50  0001 C CNN
+F 3 "" H 1550 1700 50  0001 C CNN
+	1    1550 1700
 	0    -1   -1   0
 $EndComp
@@
 L power:+12V #PWR0143
 U 1 1 5FDFF0AF
-P 1850 2100
-F 0 "#PWR0143" H 1850 1950 50  0001 C CNN
-F 1 "+12V" V 1865 2228 50  0000 L CNN
-F 2 "" H 1850 2100 50  0001 C CNN
-F 3 "" H 1850 2100 50  0001 C CNN
-	1    1850 2100
+P 1550 2100
+F 0 "#PWR0143" H 1550 1950 50  0001 C CNN
+F 1 "+12V" V 1565 2228 50  0000 L CNN
+F 2 "" H 1550 2100 50  0001 C CNN
+F 3 "" H 1550 2100 50  0001 C CNN
+	1    1550 2100
 	0    -1   -1   0
 $EndComp
-Connection ~ 1850 2100
 Wire Wire Line
 	2350 1800 2350 1900
@@
 L power:GND #PWR0156
 U 1 1 5FDFF0BB
-P 4750 1900
-F 0 "#PWR0156" H 4750 1650 50  0001 C CNN
-F 1 "GND" V 4755 1772 50  0000 R CNN
-F 2 "" H 4750 1900 50  0001 C CNN
-F 3 "" H 4750 1900 50  0001 C CNN
-	1    4750 1900
+P 5150 1900
+F 0 "#PWR0156" H 5150 1650 50  0001 C CNN
+F 1 "GND" V 5155 1772 50  0000 R CNN
+F 2 "" H 5150 1900 50  0001 C CNN
+F 3 "" H 5150 1900 50  0001 C CNN
+	1    5150 1900
 	0    -1   -1   0
 $EndComp
@@
 Connection ~ 9600 4100
 Wire Wire Line
-	9600 4100 9850 4100
+	9600 4100 9750 4100
 $Comp
 L power:GND #PWR0163
@@
 $EndComp
 Connection ~ 1950 4050
-Wire Wire Line
-	1600 4050 1950 4050
 Wire Wire Line
 	1950 4050 2150 4050
@@
 F 10 "584-ADP150AUJZ-3.3R7" H 9300 3300 50  0001 L CNN "Mouser Part Number"
 F 11 "https://www.mouser.com/Search/Refine.aspx?Keyword=584-ADP150AUJZ-3.3R7" H 9300 3200 50  0001 L CNN "Mouser Price/Stock"
+F 12 "C29149" H 8350 4000 50  0001 C CNN "LCSC Part #"
+F 13 "C29149" H 8350 4000 50  0001 C CNN "LCSC"
 	1    8350 4000
 	1    0    0    -1
@@
 F 2 "Package_TO_SOT_SMD:SOT-223" H 3300 4050 50  0001 C CNN
 F 3 "http://www.ti.com/lit/ds/symlink/lm1117.pdf" H 3300 4050 50  0001 C CNN
+F 4 "C6187" H 3300 4050 50  0001 C CNN "LCSC Part #"
+F 5 "C6187" H 3300 4050 50  0001 C CNN "LCSC"
 	1    3300 4050
 	1    0    0    -1
 $EndComp
+Wire Wire Line
+	1550 1700 1650 1700
+Wire Wire Line
+	1550 2100 1650 2100
+Connection ~ 1850 2100
+$Comp
+L power:PWR_FLAG #FLG0101
+U 1 1 611AE8C1
+P 1650 1700
+F 0 "#FLG0101" H 1650 1775 50  0001 C CNN
+F 1 "PWR_FLAG" H 1650 1873 50  0000 C CNN
+F 2 "" H 1650 1700 50  0001 C CNN
+F 3 "~" H 1650 1700 50  0001 C CNN
+	1    1650 1700
+	1    0    0    -1
+$EndComp
+Connection ~ 1650 1700
+Wire Wire Line
+	1650 1700 1850 1700
+$Comp
+L power:PWR_FLAG #FLG0102
+U 1 1 611AF2EA
+P 1650 2100
+F 0 "#FLG0102" H 1650 2175 50  0001 C CNN
+F 1 "PWR_FLAG" H 1650 2273 50  0000 C CNN
+F 2 "" H 1650 2100 50  0001 C CNN
+F 3 "~" H 1650 2100 50  0001 C CNN
+	1    1650 2100
+	-1   0    0    1
+$EndComp
+Connection ~ 1650 2100
+Wire Wire Line
+	1650 2100 1850 2100
+$Comp
+L power:GND #PWR0141
+U 1 1 5FDFF093
+P 1700 1900
+F 0 "#PWR0141" H 1700 1650 50  0001 C CNN
+F 1 "GND" V 1705 1772 50  0000 R CNN
+F 2 "" H 1700 1900 50  0001 C CNN
+F 3 "" H 1700 1900 50  0001 C CNN
+	1    1700 1900
+	0    1    1    0
+$EndComp
+Wire Wire Line
+	4750 1900 5000 1900
+$Comp
+L power:PWR_FLAG #FLG0103
+U 1 1 611B4921
+P 5000 1900
+F 0 "#FLG0103" H 5000 1975 50  0001 C CNN
+F 1 "PWR_FLAG" H 5000 2073 50  0000 C CNN
+F 2 "" H 5000 1900 50  0001 C CNN
+F 3 "~" H 5000 1900 50  0001 C CNN
+	1    5000 1900
+	1    0    0    -1
+$EndComp
+Connection ~ 5000 1900
+Wire Wire Line
+	5000 1900 5150 1900
+$Comp
+L power:PWR_FLAG #FLG0104
+U 1 1 611B8260
+P 9750 4100
+F 0 "#FLG0104" H 9750 4175 50  0001 C CNN
+F 1 "PWR_FLAG" H 9750 4273 50  0000 C CNN
+F 2 "" H 9750 4100 50  0001 C CNN
+F 3 "~" H 9750 4100 50  0001 C CNN
+	1    9750 4100
+	1    0    0    -1
+$EndComp
+Connection ~ 9750 4100
+Wire Wire Line
+	9750 4100 9850 4100
+Wire Wire Line
+	1600 4050 1950 4050
 $EndSCHEMATC

Commit message: use electrolytic caps for +/-12V rails
Parts:
- C48, C49: footprint Capacitor_SMD:C_0805_2012Metric -> Capacitor_SMD:CP_Elec_5x5.3; LCSC C45783 -> C249700; LCSC Part # C45783 -> C249700
Changed lines of the file:
@@
 F 0 "C48" V 4148 1700 50  0000 C CNN
 F 1 "22u" V 4239 1700 50  0000 C CNN
-F 2 "Capacitor_SMD:C_0805_2012Metric" H 4438 1550 50  0001 C CNN
+F 2 "Capacitor_SMD:CP_Elec_5x5.3" H 4438 1550 50  0001 C CNN
 F 3 "~" H 4400 1700 50  0001 C CNN
-F 4 "C45783" H 4400 1700 50  0001 C CNN "LCSC Part #"
-F 5 "C45783" H 4400 1700 50  0001 C CNN "LCSC"
+F 4 "C249700" H 4400 1700 50  0001 C CNN "LCSC Part #"
+F 5 "C249700" H 4400 1700 50  0001 C CNN "LCSC"
 	1    4400 1700
 	0    1    1    0
@@
 F 0 "C49" V 4148 2100 50  0000 C CNN
 F 1 "22u" V 4239 2100 50  0000 C CNN
-F 2 "Capacitor_SMD:C_0805_2012Metric" H 4438 1950 50  0001 C CNN
+F 2 "Capacitor_SMD:CP_Elec_5x5.3" H 4438 1950 50  0001 C CNN
 F 3 "~" H 4400 2100 50  0001 C CNN
-F 4 "C45783" H 4400 2100 50  0001 C CNN "LCSC Part #"
-F 5 "C45783" H 4400 2100 50  0001 C CNN "LCSC"
+F 4 "C249700" H 4400 2100 50  0001 C CNN "LCSC Part #"
+F 5 "C249700" H 4400 2100 50  0001 C CNN "LCSC"
 	1    4400 2100
 	0    1    1    0
